File: FS-VG501/FrameUnit/msx_frame_unit.sch (KiCad schematic (older format))
At the start: 113 parts, among them CN1 Conn_01x02, CN2 Conn_01x10, CN3 Conn_01x04, CN4 Conn_01x10, CN5 Conn_01x10, CN7 Conn_01x06, CN8 Conn_01x06, CN9 Conn_01x02, IC1 74LS245, IC10 74S08, IC11 74LS273, IC12 74LS273, IC13 74LS138, IC14 74LS04, IC15 74LS11, IC16 74S124/74LS629, IC17 74LS153, IC18 74LS153, IC19 74LS153, IC2 74LS244, IC20 74LS08, IC21 SLA6430, IC22 74LS32, IC23 SLA6170, IC24 TC15G008AP, IC24 TC5081AP, IC25 74HC174, IC25 TC15G008AP, IC26 74LS153, IC27 74LS153, IC27 TC15G008AP, IC28 TC15G008AP, IC3 74LS123, IC30 TC15G008AP, IC31 74HC174, IC32 74LS153, IC33 74LS153, IC36 74LS04, IC39 74LS54, IC4 74LS09, IC40 74LS54, IC41 74HC174, IC42 74LS153, IC43 74LS153, IC44 74LS04, IC45 74LS54, IC46 74LS54, IC47 DRAM_4464, IC48 DRAM_4464, IC49 DRAM_4464, IC5 MB40576, IC50 DRAM_4464, IC51 DRAM_4464, IC52 DRAM_4464, IC53 DRAM_4464, IC54 DRAM_4464, IC55 DRAM_4464, IC56 DRAM_4464, IC57 DRAM_4464, IC58 DRAM_4464, IC59 DRAM_4464, IC6 MB40576, IC60 DRAM_4464, IC61 DRAM_4464, IC62 DRAM_4464, IC63 DRAM_4464, IC64 DRAM_4464, IC65 DRAM_4464, IC66 DRAM_4464, IC67 DRAM_4164, IC68 DRAM_4164, IC69 DRAM_4164, IC7 MB40576, IC70 DRAM_4164, IC8 74LS32, IC9 74LS10

Commit message: Add files via upload
Parts:
- added IC29: 74LS32, symbol 74xx:74LS32
Connections:
- net 1_DRAM_DOUT is gone; now on net 1_Q: IC46.1, IC46.13
- net 2_DRAM_DOUT is gone; now on net 2_Q: IC45.1, IC45.13
- net 3_DRAM_DOUT is gone; now on net 3_Q: IC39.1, IC39.13
- net 4_DRAM_DOUT is gone; now on net 4_Q: IC40.1, IC40.13
- net IC30_16 is gone; now on net 2DQ3: IC45.11, IC45.2
- net IC30_22 is gone; now on net 1DQ3: IC46.11, IC46.2
- net IC30_39 is gone; now on net 3DQ2: IC39.11, IC39.2
- net IC30_45 is gone; now on net 4DQ2: IC40.11, IC40.2
- net A0_: now also IC47.14 (A0), IC48.14 (A0), IC49.14 (A0), IC50.14 (A0), IC67.13 (A6), IC68.13 (A6), IC69.13 (A6), IC70.13 (A6)
- net A1_: now also IC47.13 (A1), IC48.13 (A1), IC49.13 (A1), IC50.13 (A1), IC67.12 (A3), IC68.12 (A3), IC69.12 (A3), IC70.12 (A3)
- net A2_: now also IC47.12 (A2), IC48.12 (A2), IC49.12 (A2), IC50.12 (A2), IC67.11 (A4), IC68.11 (A4), IC69.11 (A4), IC70.11 (A4)
- net A3_: now also IC47.11 (A3), IC48.11 (A3), IC49.11 (A3), IC50.11 (A3), IC67.10 (A5), IC68.10 (A5), IC69.10 (A5), IC70.10 (A5)
- net A4_: now also IC47.8 (A4), IC48.8 (A4), IC49.8 (A4), IC50.8 (A4), IC67.7 (A1), IC68.7 (A1), IC69.7 (A1), IC70.7 (A1)
- net A5_: now also IC47.7 (A5), IC48.7 (A5), IC49.7 (A5), IC50.7 (A5), IC67.6 (A2), IC68.6 (A2), IC69.6 (A2), IC70.6 (A2)
- net A6_: now also IC47.6 (A6), IC48.6 (A6), IC49.6 (A6), IC50.6 (A6), IC67.5 (A0), IC68.5 (A0), IC69.5 (A0), IC70.5 (A0)
- net A7_: now also IC47.10 (A7), IC48.10 (A7), IC49.10 (A7), IC50.10 (A7), IC67.9 (A7), IC68.9 (A7), IC69.9 (A7), IC70.9 (A7)
- net PB_RD_: now also IC30.44 (IO), IC50.4 (W), IC29.1
- net 15_6: now reaches IC15.6, IC39.10, IC39.9, IC40.10, IC40.9, IC45.10, IC45.9, IC46.10, IC46.9
- net 2DQ3: now reaches IC30.16 (IO)
- net 2DQ3: now also IC48.15 (DQ3)
- net 1DQ3: now reaches IC30.22 (IO)
- net 1DQ3: now also IC47.15 (DQ3)
- net 5G_RAS: now reaches IC30.28 (IO)
- net 5G_RAS: now also IC47.5 (RAS), IC48.5 (RAS), IC49.5 (RAS), IC50.5 (RAS), IC67.4 (RAS), IC68.4 (RAS), IC69.4 (RAS), IC70.4 (RAS)
- net 5G_CAS: now reaches IC30.29 (IO)
- net 5G_CAS: now also IC47.16 (CAS), IC48.16 (CAS), IC49.16 (CAS), IC50.16 (CAS), IC67.15 (CAS), IC68.15 (CAS), IC69.15 (CAS), IC70.15 (CAS)
- net 3DQ2: now reaches IC30.39 (IO)
- net 3DQ2: now also IC49.3 (DQ2)
- net 4DQ2: now reaches IC30.45 (IO)
- net 4DQ2: now also IC50.3 (DQ2)
- net 4_Q: now reaches IC70.14 (Q)
- net at IC70.2 (D): now also IC50.2 (DQ1)
- net at IC70.3 (W): now also IC29.3
- net 1_Q: now reaches IC67.14 (Q)
- net at IC67.2 (D): now also IC47.17 (DQ4)
- net at IC67.3 (W): now also IC29.6
- net 2_Q: now reaches IC68.14 (Q)
- net at IC68.2 (D): now also IC48.17 (DQ4)
- net at IC68.3 (W): now also IC29.8
- net 3_Q: now reaches IC69.14 (Q)
- net at IC69.2 (D): now also IC49.2 (DQ1)
- net at IC69.3 (W): now also IC29.11
- net 5G_24: now reaches IC47.2 (DQ1)
- net 5G_25: now reaches IC47.3 (DQ2)
- net 5G_21: now reaches IC47.4 (W)
- net 5G_18: now reaches IC48.2 (DQ1)
- net 5G_19: now reaches IC48.3 (DQ2)
- net 5G_15: now reaches IC48.4 (W)
- net 5G_42: now reaches IC49.15 (DQ3)
- net 5G_41: now reaches IC49.17 (DQ4)
- net 5G_38: now reaches IC49.4 (W)
- net 5G_48: now reaches IC50.15 (DQ3)
- net 5G_47: now reaches IC50.17 (DQ4)
- net SLA6430_41: now reaches IC21.41 (GND)
- net SLA6430_41: now also IC29.10, IC29.13, IC29.2, IC29.5
- new net 5_G008_15: IC29.12
- new net 5_G008_21: IC29.4
- new net 5_G008_38: IC29.9
Other:
- moved on the sheet: IC47, IC49, IC50, IC67, IC68, IC69

Commit message: Add files via upload
Parts:
- added D?: D, symbol agg-kicad:D
- added R?: 10K, symbol agg-kicad:R
Connections:
- net 5G_15 is gone; now on net 5G_2_W: IC48.4 (W)
- net 5G_18 is gone; now on net 5G_2DQ1: IC48.2 (DQ1)
- net 5G_19 is gone; now on net 5G_2DQ2: IC48.3 (DQ2)
- net 5G_21 is gone; now on net 5G_1_W: IC47.4 (W)
- net 5G_24 is gone; now on net 5G_1DQ1: IC47.2 (DQ1)
- net 5G_25 is gone; now on net 5G_1DQ2: IC47.3 (DQ2)
- net 5G_38 is gone; now on net 5G_3_W: IC49.4 (W)
- net 5G_41 is gone; now on net 5G_3DQ4: IC49.17 (DQ4)
- net 5G_42 is gone; now on net 5G_3DQ3: IC49.15 (DQ3)
- net 5G_47 is gone; now on net 5G_4DQ4: IC50.17 (DQ4)
- net 5G_48 is gone; now on net 5G_4DQ3: IC50.15 (DQ3)
- net 5_G008_15 is gone; now on net 5G_2_W: IC29.12
- net 5_G008_21 is gone; now on net 5G_1_W: IC29.4
- net 5_G008_38 is gone; now on net 5G_3_W: IC29.9
- net +5V: now also R?.1
- net 1DQ3: no longer IC30.22 (IO), IC47.15 (DQ3)
- net 2DQ3: no longer IC30.16 (IO), IC48.15 (DQ3)
- net 3DQ2: no longer IC30.39 (IO), IC49.3 (DQ2)
- net 4DQ2: no longer IC30.45 (IO), IC50.3 (DQ2)
- net A6: now also IC23.34 (IO)
- net CN5_3: now also D?.1
- net GND: now also IC23.1 (GND), IC23.32 (GND), IC23.35 (GND), IC23.4 (GND), IC23.40 (GND), IC24.1 (GND), IC24.20 (GND), IC24.27 (GND), IC24.32 (GND), IC24.43 (GND), IC24.53 (GND), IC25.1 (GND), IC25.20 (GND), IC25.27 (GND), IC25.32 (GND), IC25.43 (GND), IC25.53 (GND), IC25.58 (IO), IC27.1 (GND), IC27.20 (GND), IC27.27 (GND), IC27.32 (GND), IC27.43 (GND), IC27.53 (GND), IC28.1 (GND), IC28.20 (GND), IC28.27 (GND), IC28.32 (GND), IC28.43 (GND), IC28.53 (GND), IC30.1 (GND), IC30.20 (GND), IC30.27 (GND), IC30.32 (GND), IC30.43 (GND), IC30.53 (GND), IC47.1 (G), IC47.18 (GND), IC48.1 (G), IC48.18 (GND), IC49.18 (GND), IC50.18 (GND), IC67.16 (GND), IC68.16 (GND), IC69.16 (GND), IC70.16 (GND)
- net SLA6170_60: now reaches IC14.3, IC23.60 (IO)
- net SLA6170_60: now also IC25.63 (IO), IC28.63 (IO), IC30.63 (IO)
- net SLA6170_49: now reaches IC24.10 (IO)
- net SLA6170_49: now also IC23.49 (IO), IC25.10 (IO), IC27.10 (IO), IC28.10 (IO), IC30.10 (IO)
- net SLA6170_50: now reaches IC24.11 (IO)
- net SLA6170_50: now also IC23.50 (IO), IC25.11 (IO), IC27.11 (IO), IC28.11 (IO), IC30.11 (IO)
- net SLA6170_51: now reaches IC24.12 (IO)
- net SLA6170_51: now also IC23.51 (IO), IC25.12 (IO), IC27.12 (IO), IC28.12 (IO), IC30.12 (IO)
- net SLA6430_60: now reaches IC24.13 (IO)
- net SLA6430_60: now also IC21.60 (IO), IC25.13 (IO), IC27.13 (IO), IC28.13 (IO), IC30.13 (IO)
- net at IC24.14 (IO), IC25.14 (IO), IC27.14 (IO)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: now also IC30.14 (IO)
- net 1G_2_W: now reaches IC24.15 (IO)
- net 1G_2DQ3: now reaches IC24.16 (IO)
- net 1G_2DQ3: now also IC52.15 (DQ3)
- net 1G_2DQ4: now reaches IC24.17 (IO)
- net 1G_2DQ4: now also IC52.17 (DQ4)
- net 1G_2DQ1: now reaches IC24.18 (IO)
- net 1G_2DQ1: now also IC52.2 (DQ1)
- net 1G_2DQ2: now reaches IC24.19 (IO)
- net 1G_2DQ2: now also IC52.3 (DQ2)
- net 1G_1_W: now reaches IC24.21 (IO)
- net 1G_1_W: now also IC51.4 (W), IC52.4 (W)
- net 1G_1DQ3: now reaches IC24.22 (IO)
- net 1G_1DQ3: now also IC51.15 (DQ3)
- net 1G_1DQ4: now reaches IC24.23 (IO)
- net 1G_1DQ4: now also IC51.17 (DQ4)
- net 1G_1DQ1: now reaches IC24.24 (IO)
- net 1G_1DQ1: now also IC51.2 (DQ1)
- net 1G_1DQ2: now reaches IC24.25 (IO)
- net 1G_1DQ2: now also IC51.3 (DQ2)
- net SLA6430_40: now reaches IC24.26 (IO)
- net SLA6430_40: now also IC21.40 (GND), IC23.36 (IO), IC27.26 (IO), IC28.26 (IO), IC30.26 (IO)
- net 1G_RAS: now reaches IC24.28 (IO)
- net 1G_RAS: now also IC51.5 (RAS), IC52.5 (RAS), IC53.5 (RAS), IC54.5 (RAS)
- net 1G_CAS: now reaches IC24.29 (IO)
- net 1G_CAS: now also IC51.16 (CAS), IC52.16 (CAS), IC53.16 (CAS), IC54.16 (CAS)
- net 1G_3_W: now reaches IC24.38 (IO)
- net 1G_3_W: now also IC53.4 (W)
- net 1G_3DQ2: now reaches IC24.39 (IO)
- net 1G_3DQ2: now also IC25.39 (IO), IC53.3 (DQ2)
- net 1G_3DQ1: now reaches IC24.40 (IO)
- net 1G_3DQ1: now also IC25.40 (IO), IC53.2 (DQ1)
- net 1G_3DQ4: now reaches IC24.41 (IO)
- net 1G_3DQ4: now also IC53.17 (DQ4)
- net 1G_3DQ3: now reaches IC24.42 (IO)
- net 1G_3DQ3: now also IC53.15 (DQ3)
- net 1G_4_W: now reaches IC24.44 (IO)
- net 1G_4_W: now also IC54.4 (W)
- net 1G_4DQ2: now reaches IC24.45 (IO)
- net 1G_4DQ2: now also IC54.3 (DQ2)
- net 1G_4DQ1: now reaches IC24.46 (IO)
- net 1G_4DQ1: now also IC54.2 (DQ1)
- net 1G_4DQ4: now reaches IC24.47 (IO)
- net 1G_4DQ4: now also IC54.17 (DQ4)
- net 1G_4DQ3: now reaches IC24.48 (IO)
- net 1G_4DQ3: now also IC54.15 (DQ3)
- net SLA6430_71: now reaches IC24.56 (IO)
- net SLA6430_71: now also IC21.71 (IO), IC25.56 (IO), IC27.56 (IO), IC28.56 (IO), IC30.56 (IO)
- net SLA6430_70: now reaches IC24.57 (IO)
- net SLA6430_70: now also IC21.70 (IO), IC25.57 (IO), IC27.57 (IO), IC28.57 (IO), IC30.57 (IO)
- net SLA6170_53: now reaches IC24.58 (IO)
- net SLA6170_53: now also IC23.53 (IO)
- net SLA6170_52: now reaches IC24.59 (IO)
- net SLA6170_52: now also IC23.52 (IO), IC25.59 (IO), IC27.59 (IO), IC28.59 (IO), IC30.59 (IO)
- net SLA6430_78: now reaches IC24.6 (IO)
- net SLA6430_78: now also IC21.78 (IO), IC27.6 (IO), IC28.6 (IO)
- net SLA6430_77: now reaches IC24.7 (IO)
- net SLA6430_77: now also IC21.77 (IO), IC27.7 (IO), IC28.7 (IO)
- net SLA6430_76: now reaches IC24.8 (IO)
- net SLA6430_76: now also IC21.76 (IO), IC27.8 (IO), IC30.8 (IO)
- net SLA6430_75: now reaches IC24.9 (IO)
- net SLA6430_75: now also IC21.75 (IO), IC27.9 (IO), IC30.9 (IO)
- net 2G_2_W: now reaches IC25.15 (IO)
- net 2G_2_W: now also IC56.4 (W)
- net 2G_2DQ3: now reaches IC25.16 (IO)
- net 2G_2DQ3: now also IC56.15 (DQ3)
- net 2G_2DQ4: now reaches IC25.17 (IO)
- net 2G_2DQ4: now also IC56.17 (DQ4)
- net 2G_2DQ1: now reaches IC25.18 (IO)
- net 2G_2DQ1: now also IC56.2 (DQ1)
- net 2G_2DQ2: now reaches IC25.19 (IO)
- net 2G_2DQ2: now also IC56.3 (DQ2)
- net 2G_1_W: now reaches IC25.21 (IO)
- net 2G_1_W: now also IC55.4 (W)
- net 2G_1DQ3: now reaches IC25.22 (IO)
- net 2G_1DQ3: now also IC55.15 (DQ3)
- net 2G_1DQ4: now reaches IC25.23 (IO)
- net 2G_1DQ4: now also IC55.17 (DQ4)
- net 2G_1DQ1: now reaches IC25.24 (IO)
- net 2G_1DQ1: now also IC55.2 (DQ1)
- net 2G_1DQ2: now reaches IC25.25 (IO)
- net 2G_1DQ2: now also IC55.3 (DQ2)
- net 2G_RAS: now reaches IC25.28 (IO)
- net 2G_RAS: now also IC55.5 (RAS), IC56.5 (RAS), IC57.5 (RAS), IC58.5 (RAS)
- net 2G_CAS: now reaches IC25.29 (IO)
- net 2G_CAS: now also IC55.16 (CAS), IC56.16 (CAS), IC57.16 (CAS), IC58.16 (CAS)
- net 2G_3_W: now reaches IC25.38 (IO)
- net 2G_3DQ4: now reaches IC25.41 (IO)
- net 2G_3DQ4: now also IC57.17 (DQ4)
- net 2G_3DQ3: now reaches IC25.42 (IO)
- net 2G_3DQ3: now also IC57.15 (DQ3)
- net 2G_4_W: now reaches IC25.44 (IO)
- net 2G_4DQ2: now reaches IC25.45 (IO)
- net 2G_4DQ2: now also IC58.3 (DQ2)
- net 2G_4DQ1: now reaches IC25.46 (IO)
- net 2G_4DQ1: now also IC58.2 (DQ1)
- net 2G_4DQ4: now reaches IC25.47 (IO)
- net 2G_4DQ4: now also IC58.17 (DQ4)
- net 2G_4DQ3: now reaches IC25.48 (IO)
- net 2G_4DQ3: now also IC58.15 (DQ3)
- net SLA6430_62: now reaches IC25.55 (IO)
- net SLA6430_62: now also IC21.62 (IO), IC27.55 (IO), IC28.55 (IO), IC30.55 (IO)
- net SLA6170_56: now reaches IC25.60 (IO)
- net SLA6170_56: now also IC23.56 (IO), IC28.60 (IO), IC30.60 (IO)
- net SLA6170_58: now reaches IC25.61 (IO)
- net SLA6170_58: now also IC23.58 (IO), IC28.61 (IO), IC30.61 (IO)
- net SLA6170_59: now reaches IC25.62 (IO)
- net SLA6170_59: now also IC23.59 (IO), IC28.62 (IO), IC30.62 (IO)
- net 3G_2_W: now reaches IC27.15 (IO)
- net 3G_2_W: now also IC60.4 (W)
- net 3G_2DQ3: now reaches IC27.16 (IO)
- net 3G_2DQ3: now also IC60.15 (DQ3)
- net 3G_2DQ4: now reaches IC27.17 (IO)
- net 3G_2DQ4: now also IC60.17 (DQ4)
- net 3G_2DQ1: now reaches IC27.18 (IO)
- net 3G_2DQ1: now also IC60.2 (DQ1)
- net 3G_2DQ2: now reaches IC27.19 (IO)
- net 3G_2DQ2: now also IC60.3 (DQ2)
- net 3G_1_W: now reaches IC27.21 (IO)
- net 3G_1_W: now also IC59.4 (W)
- net 3G_1DQ3: now reaches IC27.22 (IO)
- net 3G_1DQ3: now also IC59.15 (DQ3)
- net 3G_1DQ4: now reaches IC27.23 (IO)
- net 3G_1DQ4: now also IC59.17 (DQ4)
- net 3G_1DQ1: now reaches IC27.24 (IO)
- net 3G_1DQ1: now also IC59.2 (DQ1)
- net 3G_1DQ2: now reaches IC27.25 (IO)
- net 3G_1DQ2: now also IC59.3 (DQ2)
- net 3G_RAS: now reaches IC27.28 (IO)
- net 3G_RAS: now also IC59.5 (RAS), IC60.5 (RAS), IC61.5 (RAS), IC62.5 (RAS)
- net 3G_CAS: now reaches IC27.29 (IO)
- net 3G_CAS: now also IC59.16 (CAS), IC60.16 (CAS), IC61.16 (CAS), IC62.16 (CAS)
- net 3G_3_W: now reaches IC27.38 (IO)
- net 3G_3_W: now also IC61.4 (W)
- net 3G_3DQ2: now reaches IC27.39 (IO)
- net 3G_3DQ2: now also IC61.3 (DQ2)
- net 3G_3DQ1: now reaches IC27.40 (IO)
- net 3G_3DQ1: now also IC61.2 (DQ1)
- net 3G_3DQ4: now reaches IC27.41 (IO)
- net 3G_3DQ4: now also IC61.17 (DQ4)
- net 3G_3DQ3: now reaches IC27.42 (IO)
- net 3G_3DQ3: now also IC61.15 (DQ3)
- net 3G_4_W: now reaches IC27.44 (IO)
- net 3G_4_W: now also IC62.4 (W)
- net 3G_4DQ2: now reaches IC27.45 (IO)
- net 3G_4DQ2: now also IC62.3 (DQ2)
- net 3G_4DQ1: now reaches IC27.46 (IO)
- net 3G_4DQ1: now also IC62.2 (DQ1)
- net 3G_4DQ4: now reaches IC27.47 (IO)
- net 3G_4DQ4: now also IC62.17 (DQ4)
- net 3G_4DQ3: now reaches IC27.48 (IO)
- net 3G_4DQ3: now also IC62.15 (DQ3)
- net SLA6430_67: now reaches IC27.54 (IO)
- net SLA6430_67: now also IC21.67 (IO)
- net SLA6170_54: now reaches IC27.58 (IO)
- net SLA6170_54: now also IC23.54 (IO)
- net 4G_2_W: now reaches IC28.15 (IO)
- net 4G_2_W: now also IC64.4 (W)
- net 4G_2DQ3: now reaches IC28.16 (IO)
- net 4G_2DQ3: now also IC64.15 (DQ3)
- net 4G_2DQ4: now reaches IC28.17 (IO)
- net 4G_2DQ4: now also IC64.17 (DQ4)
- net 4G_2DQ1: now reaches IC28.18 (IO)
- net 4G_2DQ1: now also IC64.2 (DQ1)
- net 4G_2DQ2: now reaches IC28.19 (IO)
- net 4G_2DQ2: now also IC64.3 (DQ2)
- net 4G_1_W: now reaches IC28.21 (IO)
- net 4G_1_W: now also IC63.4 (W)
- net 4G_1DQ3: now reaches IC28.22 (IO)
- net 4G_1DQ3: now also IC63.15 (DQ3)
- net 4G_1DQ4: now reaches IC28.23 (IO)
- net 4G_1DQ4: now also IC63.17 (DQ4)
- net 4G_1DQ1: now reaches IC28.24 (IO)
- net 4G_1DQ1: now also IC63.2 (DQ1)
- net 4G_1DQ2: now reaches IC28.25 (IO)
- net 4G_1DQ2: now also IC63.3 (DQ2)
- net 4G_RAS: now reaches IC28.28 (IO)
- net 4G_RAS: now also IC63.5 (RAS), IC64.5 (RAS), IC65.5 (RAS), IC66.5 (RAS)
- net 4G_CAS: now reaches IC28.29 (IO)
- net 4G_CAS: now also IC63.16 (CAS), IC64.16 (CAS), IC65.16 (CAS), IC66.16 (CAS)
- net 4G_3_W: now reaches IC28.38 (IO)
- net 4G_3_W: now also IC65.4 (W)
- net 4G_3DQ2: now reaches IC28.39 (IO)
- net 4G_3DQ2: now also IC65.3 (DQ2)
- net 4G_3DQ1: now reaches IC28.40 (IO)
- net 4G_3DQ1: now also IC65.2 (DQ1)
- net 4G_3DQ4: now reaches IC28.41 (IO)
- net 4G_3DQ4: now also IC65.17 (DQ4)
- net 4G_3DQ3: now reaches IC28.42 (IO)
- net 4G_3DQ3: now also IC65.15 (DQ3)
- net 4G_4_W: now reaches IC28.44 (IO)
- net 4G_4_W: now also IC66.4 (W)
- net 4G_4DQ2: now reaches IC28.45 (IO)
- net 4G_4DQ2: now also IC66.3 (DQ2)
- net 4G_4DQ1: now reaches IC28.46 (IO)
- net 4G_4DQ1: now also IC66.2 (DQ1)
- net 4G_4DQ4: now reaches IC28.47 (IO)
- net 4G_4DQ4: now also IC66.17 (DQ4)
- net 4G_4DQ3: now reaches IC28.48 (IO)
- net 4G_4DQ3: now also IC66.15 (DQ3)
- net SLA6430_66: now reaches IC28.54 (IO)
- net SLA6430_66: now also IC21.66 (IO), IC30.54 (IO)
- net SLA6170_55: now reaches IC28.58 (IO)
- net SLA6170_55: now also IC23.55 (IO), IC30.58 (IO)
- net SLA6430_80: now reaches IC28.8 (IO)
- net SLA6430_80: now also IC21.80 (VCC)
- net SLA6430_79: now reaches IC28.9 (IO)
- net SLA6430_79: now also IC21.79 (IO)
- net 5G_2_W: now reaches IC30.15 (IO)
- net 5G_2DQ4: now reaches IC30.17 (IO)
- net 5G_2DQ4: now also IC48.17 (DQ4), IC68.2 (D)
- net 5G_2DQ1: now reaches IC30.18 (IO)
- net 5G_2DQ2: now reaches IC30.19 (IO)
- net 5G_1_W: now reaches IC30.21 (IO)
- net 5G_1DQ4: now reaches IC30.23 (IO)
- net 5G_1DQ4: now also IC47.17 (DQ4), IC67.2 (D)
- net 5G_1DQ1: now reaches IC30.24 (IO)
- net 5G_1DQ2: now reaches IC30.25 (IO)
- net 5G_3_W: now reaches IC30.38 (IO)
- net 5G_3DQ1: now reaches IC30.40 (IO)
- net 5G_3DQ1: now also IC49.2 (DQ1), IC69.2 (D)
- net 5G_3DQ4: now reaches IC30.41 (IO)
- net 5G_3DQ3: now reaches IC30.42 (IO)
- net 5G_4DQ1: now reaches IC30.46 (IO)
- net 5G_4DQ1: now also IC50.2 (DQ1), IC70.2 (D)
- net 5G_4DQ4: now reaches IC30.47 (IO)
- net 5G_4DQ3: now reaches IC30.48 (IO)
- net SLA6430_74: now reaches IC30.6 (IO)
- net SLA6430_74: now also IC21.74 (IO)
- net SLA6430_73: now reaches IC30.7 (IO)
- net SLA6430_73: now also IC21.73 (IO)
- net SLA6430_43: now reaches IC23.37 (IO)
- net SLA6430_43: now also IC21.43 (IO)
- net at IC23.41 (IO): now also D?.2, R?.2
- net SLA6430_22: now reaches IC23.42 (IO)
- net SLA6430_22: now also IC21.22 (IO)
- net SLA6430_21: now reaches IC23.43 (IO)
- net SLA6430_21: now also IC21.21 (IO)
- net SLA6430_19: now reaches IC23.44 (IO)
- net SLA6430_19: now also IC21.19 (IO)
- net SLA6430_20: now reaches IC23.45 (IO)
- net SLA6430_20: now also IC21.20 (IO)
- net SLA6430_18: now reaches IC23.46 (IO)
- net SLA6430_18: now also IC21.18 (IO)
- net 2G_44: now reaches IC58.4 (W)
- net 2G_3DQ1: now reaches IC57.2 (DQ1)
- net 2G_3DQ2: now reaches IC57.3 (DQ2)
- net 2G_38: now reaches IC57.4 (W)
- net SLA6430_64: now reaches IC21.64 (GND)
- net SLA6430_65: now reaches IC21.65 (VCC)
- net SLA6430_68: now reaches IC21.68 (IO)
- new net 5G_1DQ3: IC30.22 (IO), IC47.15 (DQ3)
- new net 5G_2DQ3: IC30.16 (IO), IC48.15 (DQ3)
- new net 5G_3DQ2: IC30.39 (IO), IC49.3 (DQ2)
- new net 5G_4DQ2: IC30.45 (IO), IC50.3 (DQ2)
Other:
- moved on the sheet: IC22A, IC36F, IC48, IC49, IC50, IC51, IC52, IC53, IC54, IC55, IC56, IC57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

Commit message: Add files via upload
Parts:
- added C119, C50, C51, C57, C58, C59, C72, C74, TC1: C, symbol agg-kicad:C
- added D2, D5, D6: D, symbol agg-kicad:D
- added IC28: 74LS123, symbol 74xx:74LS123
- added unit 2 of IC28
- added R22: 1K, symbol agg-kicad:R
- added R23: 915K, symbol agg-kicad:R
- added R24, R25: 2K, symbol agg-kicad:R
- added R26, R29: 48K, symbol agg-kicad:R
- added R27: 22K, symbol agg-kicad:R
- added R28: 150K, symbol agg-kicad:R
- added R39: 25K, symbol agg-kicad:R
- added R63, R64: 2K2, symbol agg-kicad:R
- added R?: 5K6, symbol agg-kicad:R
- added VR1: 6K2, symbol agg-kicad:R
- R1: renamed from R?; value R -> 7K
- R2: renamed from R?; value R -> 20K
- R58: renamed from R?; value R -> 7K1
- gave numbers to parts that had none: 5
Connections:
- net CN4_8 is gone; now on net SLA6430_48: CN4.8 (Pin_8)
- net CN4_9 is gone; now on net SLA6170_22: CN4.9 (Pin_9)
- net CN5_4 is gone; now on net SLA6170_26: CN5.4 (Pin_4)
- net CN5_5 is gone; now on net SLA6170_27: CN5.5 (Pin_5)
- net CN5_6 is gone; now on net SLA6170_30: CN5.6 (Pin_6)
- net +5V: now also IC16.6 (EN), IC24.5 (Vdd), IC30.64 (VCC), IC31.16 (VCC), C57.1, D2.1, IC28.10 (B), IC28.11 (Clr), IC28.2 (B), IC28.3 (Clr), R22.1, R25.1, R27.2, R39.1, R63.2, R64.1, R?.2, VR1.1
- net CN2_1: now also CN2.1 (Pin_1)
- net CN2_10: now also CN2.10 (Pin_10)
- net CN2_5: now also CN2.5 (Pin_5)
- net CN2_7: now also CN2.7 (Pin_7)
- net CN2_8: now also CN2.8 (Pin_8)
- net CN2_9: now also CN2.9 (Pin_9)
- net CN3_2: now also CN3.2 (Pin_2), R?.2
- net CN3_3: now also CN3.3 (Pin_3), R?.2
- net CN3_4: now also CN3.4 (Pin_4), R?.2
- net D7: now also D5.2
- net GND: now also IC16.11 (EN), IC16.3 (RNG), IC51.18 (GND), IC52.18 (GND), IC53.18 (GND), IC54.18 (GND), IC55.18 (GND), IC56.18 (GND), IC57.18 (GND), IC58.18 (GND), IC59.18 (GND), IC60.18 (GND), IC61.18 (GND), IC62.18 (GND), IC63.18 (GND), IC64.18 (GND), IC65.18 (GND), IC66.18 (GND), C119.2, C51.2, C57.2, C58.1, C72.2, C74.2, IC28.14 (Cext), IC28.6 (Cext), R24.2
- net PB_RD_: now also IC28.1 (A)
- net SLA6170_29: now also IC23.29 (IO), C119.1
- net SLA6170_60: now also R63.1, R64.2
- net SLA6430_41: now also R?.1
- net SLA6430_43: now also D2.2, R27.1
- net SLA6430_48: no longer IC9.3
- net SLA6430_49: now also IC9.3; no longer IC9.11
- net SLA6170_19: now reaches CN2.2 (Pin_2)
- net SLA6170_19: now also IC23.19 (IO)
- net SLA6170_20: now reaches CN2.3 (Pin_3)
- net SLA6170_20: now also IC23.20 (IO)
- net at IC16.1 (FC): now also R26.1
- net SLA6170_63: now reaches IC16.10 (Y)
- net at IC16.12 (CX2): now also C50.2, TC1.2
- net at IC16.13 (CX1): now also C50.1, TC1.1
- net at IC16.14 (RNG): now also C51.1, R24.1, R25.2
- net at IC24.1 (Aout): now also C59.1, R26.2
- net at IC24.2 (Ain): now also C58.2, R29.2
- net at IC24.3 (PDout): now also R28.1, R29.1
- net at IC24.7 (S): now also IC28.12 (~Q)
- net at 21477.2.2, IC23.2 (IO): now also R23.2
- net SLA6170_22: now reaches IC23.22 (IO)
- net SLA6170_22: now also D6.2
- net SLA6170_26: now reaches IC23.26 (IO)
- net SLA6170_27: now reaches IC23.27 (IO)
- net SLA6170_27: now also IC28.9 (A)
- net at 21477.2.1, IC23.3 (IO): now also R23.1
- net SLA6170_30: now reaches IC23.30 (IO)
- net SLA6430_50: now reaches IC21.50 (IO)
- net SLA6430_50: now also IC9.11
- new net: D5.1, D6.1, IC28.13 (Q)
- new net: C74.1, IC28.15 (RCext), R39.2
- new net: C72.1, IC28.7 (RCext), VR1.2
- new net: C59.2, R28.2
- no-connect marks 10 -> 13
Other:
- moved on the sheet: CN5, CN8, D4, IC14B, IC16A, IC16B, IC22A, IC24, IC36A, IC36B, IC36C, IC36D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

Commit message: Add files via upload
Parts:
- removed R?: 44R, symbol agg-kicad:R
- added C1, C2, C3, C4, C5, C6: 2.2nF, symbol agg-kicad:C
- added C10, C11, C12, C13, C14, C7, C8, C9: 1nF, symbol agg-kicad:C
- added C116: 220uF/6.3V, symbol Device:CP
- added C15,C16,C18,C20-C39,C41-C44,C47,C51,C52,C55-C57,C62-C71,C73,C75,C77,C78,C80-C89,C91-C114,C117,C118: 100nF/25v, symbol agg-kicad:C
- added C45,C48,C49,C53,C60: 2200uF/6.3V, symbol Device:CP
- added C54: 22uF/6.3V, symbol Device:CP
- added C61: 470uF/16V, symbol Device:CP
- added C76, C79, C90: 47pF, symbol agg-kicad:C
- added unit 5 of IC22
- added unit 3 of IC28
- added unit 7 of IC36
- added unit 2 of IC40
- added unit 7 of IC44
- added unit 2 of IC45
- added unit 2 of IC46
- added IR11, IR21, IR31: 5K, symbol agg-kicad:R
- added IR12, IR22, IR32, R31, R40, R47: 10K, symbol agg-kicad:R
- added IR13, IR23, IR33: 20K, symbol agg-kicad:R
- added IR14, IR24, IR34: 40K, symbol agg-kicad:R
- added IR15, IR25, IR35: 80K, symbol agg-kicad:R
- added Q1, Q15, Q17, Q19, Q2, Q3, Q4, Q5, Q6, Q7, Q8: A564_PNP, symbol Device:Q_PNP_ECB
- added Q10, Q11, Q12, Q13, Q14, Q16, Q18, Q9: C1684_NPN, symbol Device:Q_NPN_ECB
- added R10, R11, R9: 680R, symbol agg-kicad:R
- added R12: 800R, symbol agg-kicad:R
- added R13, R15, R17: 2K2, symbol agg-kicad:R
- added R14, R18: 7K, symbol agg-kicad:R
- added R16, R6: 7K1, symbol agg-kicad:R
- added R19: 1K5, symbol agg-kicad:R
- added R20: 3K36, symbol agg-kicad:R
- added R21, R7: 1K17, symbol agg-kicad:R
- added R3, R33, R4, R42, R49, R5: 560R, symbol agg-kicad:R
- added R32, R41, R48: 150K, symbol agg-kicad:R
- added R34, R35, R43, R44, R50, R51: 630R, symbol agg-kicad:R
- added R36, R37, R45, R46, R52, R53: 1K8, symbol agg-kicad:R
- added R8: 209R, symbol agg-kicad:R
- added R? (x8): 1K, symbol agg-kicad:R
- added R? (x6): 470R, symbol agg-kicad:R
- added R?: R, symbol agg-kicad:R
- C119: value C -> 5.6nF
- C17: value C -> 330pF
- C19, C72, C74: value C -> 1nF
- C50: value C -> 10pF
- C51, C57, C59: value C -> 100nF
- C58: value C -> 3.3nF
- gave numbers to parts that had none: 11
Connections:
- net CN4_4 is gone; now on net SLA6170_19: CN4.4 (Pin_4)
- net CN4_5 is gone; now on net SLA6170_20: CN4.5 (Pin_5)
- net CN5_8 is gone; now on net SLA6170_28: CN5.8 (Pin_8)
- net GND is gone; now on net +5VA: C119.2, C17.2, C19.2, C51.2, C57.2, C58.1, C72.2, C74.2, CN1.1 (Pin_1), CN2.6 (Pin_6), CN4.10 (Pin_10), CN4.7 (Pin_7), CN5.10 (Pin_10), CN5.2 (Pin_2), CN5.7 (Pin_7), CN7.2 (Pin_2), CN7.4 (Pin_4), CN7.6 (Pin_6), CN8.2 (Pin_2), CN8.4 (Pin_4), CN8.6 (Pin_6), IC1.10 (GND), IC11.10 (GND), IC12.10 (GND), IC13.8 (GND), IC16.11 (EN), IC16.3 (RNG), IC17.8 (GND), IC18.8 (GND), IC19.15 (Eb), IC19.8 (GND), IC2.1 (OEa), IC2.10 (GND), IC2.17 (I3b), IC2.19 (OEb), IC2.2 (I0a), IC21.12 (IO), IC21.28 (IO), IC21.38 (IO), IC22.2, IC23.1 (GND), IC23.32 (GND), IC23.35 (GND), IC23.4 (GND), IC23.40 (GND), IC24.1 (GND), IC24.20 (GND), IC24.27 (GND), IC24.32 (GND), IC24.43 (GND), IC24.53 (GND), IC24.9 (GND), IC25.1 (GND), IC25.20 (GND), IC25.27 (GND), IC25.32 (GND), IC25.43 (GND), IC25.53 (GND), IC25.58 (IO), IC25.8 (GND), IC27.1 (GND), IC27.20 (GND), IC27.27 (GND), IC27.32 (GND), IC27.43 (GND), IC27.53 (GND), IC28.1 (GND), IC28.14 (Cext), IC28.20 (GND), IC28.27 (GND), IC28.32 (GND), IC28.43 (GND), IC28.53 (GND), IC28.6 (Cext), IC3.14 (Cext), IC3.6 (Cext), IC30.1 (GND), IC30.20 (GND), IC30.27 (GND), IC30.32 (GND), IC30.43 (GND), IC30.53 (GND), IC31.8 (GND), IC39.3, IC39.4, IC39.5, IC40.3, IC40.4, IC40.5, IC41.8 (GND), IC45.3, IC45.4, IC45.5, IC46.3, IC46.4, IC46.5, IC47.1 (G), IC47.18 (GND), IC48.1 (G), IC48.18 (GND), IC49.18 (GND), IC5.8 (GND), IC50.18 (GND), IC51.18 (GND), IC52.18 (GND), IC53.18 (GND), IC54.18 (GND), IC55.18 (GND), IC56.18 (GND), IC57.18 (GND), IC58.18 (GND), IC59.18 (GND), IC6.8 (GND), IC60.18 (GND), IC61.18 (GND), IC62.18 (GND), IC63.18 (GND), IC64.18 (GND), IC65.18 (GND), IC66.18 (GND), IC67.16 (GND), IC68.16 (GND), IC69.16 (GND), IC7.8 (GND), IC70.16 (GND), R24.2
- net +12V: now also Q10.2 (C), Q11.2 (C), Q12.2 (C), Q9.2 (C), R14.1, R16.1, R18.1, R6.1
- net +5V: now also IC10.14 (VCC), IC14.14 (VCC), IC15.14 (VCC), IC16.16 (VCC), IC17.16 (VCC), IC18.16 (VCC), IC19.16 (VCC), IC20.14 (VCC), IC23.33 (VCC), IC23.38 (VCC), IC23.39 (VCC), IC23.64 (VCC), IC24.33 (VCC), IC24.64 (VCC), IC25.16 (VCC), IC25.33 (VCC), IC25.64 (VCC), IC26.16 (VCC), IC27.16 (VCC), IC27.33 (VCC), IC27.64 (VCC), IC28.33 (VCC), IC28.64 (VCC), IC29.14 (VCC), IC3.16 (VCC), IC30.33 (VCC), IC32.16 (VCC), IC33.16 (VCC), IC39.14 (VCC), IC4.14 (VCC), IC42.16 (VCC), IC43.16 (VCC), IC47.9 (VCC), IC48.9 (VCC), IC49.9 (VCC), IC50.9 (VCC), IC51.9 (VCC), IC52.9 (VCC), IC53.9 (VCC), IC54.9 (VCC), IC55.9 (VCC), IC56.9 (VCC), IC57.9 (VCC), IC58.9 (VCC), IC59.9 (VCC), IC60.9 (VCC), IC61.9 (VCC), IC62.9 (VCC), IC63.9 (VCC), IC64.9 (VCC), IC65.9 (VCC), IC66.9 (VCC), IC67.8 (VCC), IC68.8 (VCC), IC69.8 (VCC), IC70.8 (VCC), IC8.14 (VCC), IC9.14 (VCC), C116.1, C15,C16,C18,C20-C39,C41-C44,C47,C51,C52,C55-C57,C62-C71,C73,C75,C77,C78,C80-C89,C91-C114,C117,C118.1, C45,C48,C49,C53,C60.1, C54.1, C61.1, IC22.14 (VCC), IC28.16 (VCC), IC36.14 (VCC), IC40.14 (VCC), IC44.14 (VCC), IC45.14 (VCC), IC46.14 (VCC), R?.1, R?.1, R?.1, R?.1, R?.1, R?.1, R?.1, R?.1, R?.1, R?.1, R?.1, R?.1, R?.1, R?.1, R?.1
- net 1_AD0: no longer IC41.3 (D0), IC42.7 (Za), R?.2
- net 1_AD1: no longer IC41.4 (D1), IC43.9 (Zb), R?.2
- net 1_AD2: no longer IC33.9 (Zb), IC41.6 (D2), R?.2
- net 1_AD3: no longer IC33.7 (Za), IC41.11 (D3), R?.2
- net 1_AD4: no longer IC41.13 (D4), IC43.7 (Za), R?.2
- net 1_AD5: no longer IC41.14 (D5), IC42.9 (Zb), R?.2
- net 2_AD0: no longer IC31.3 (D0), IC32.7 (Za), R?.2
- net 2_AD1: no longer IC27.9 (Zb), R?.2
- net 2_AD2: no longer IC26.9 (Zb), IC31.6 (D2), R?.2
- net 2_AD3: no longer IC26.7 (Za), IC31.11 (D3), R?.2
- net 2_AD4: no longer IC27.7 (Za), IC31.13 (D4), R?.2
- net 2_AD5: no longer IC31.14 (D5), IC32.9 (Zb), R?.2
- net 3_AD0: no longer IC19.7 (Za), IC25.3 (D0), R?.2
- net 3_AD1: no longer IC18.9 (Zb), IC25.4 (D1), R?.2
- net 3_AD2: no longer IC17.9 (Zb), IC25.6 (D2), R?.2
- net 3_AD3: no longer IC17.7 (Za), IC25.11 (D3), R?.2
- net 3_AD4: no longer IC18.7 (Za), IC25.13 (D4), R?.2
- net 3_AD5: no longer IC19.9 (Zb), IC25.14 (D5), R?.2
- net DA_CLK: now also R22.2
- net P1: now also C13.1, R?.2
- net P10_WR_: now also C6.1, R?.2
- net P11_RD_: now also C2.1, R?.2
- net P12_A0: now also C5.1, R?.2
- net P13_A1: now also C3.1, R?.2
- net P14: now also C4.1, R?.2
- net P2: now also C14.1, R?.2
- net P3: now also C11.1, R?.2
- net P4: now also C12.1, R?.2
- net P5: now also C9.1, R?.2
- net P6: now also C10.1, R?.2
- net P7: now also C7.1, R?.2
- net P8: now also C8.1, R?.2
- net P9: now also C1.1, R?.2
- net SLA6170_56: now also IC24.60 (IO), IC27.60 (IO)
- net SLA6170_58: now also IC24.61 (IO), IC27.61 (IO)
- net SLA6170_59: now also IC24.62 (IO), IC27.62 (IO)
- net SLA6170_60: now also IC24.63 (IO), IC27.63 (IO)
- net SLA6430_62: now also IC24.55 (IO)
- net SLA6430_64: now also IC25.54 (IO)
- net SLA6430_68: now also IC24.54 (IO)
- net SLA6430_73: now also IC25.9 (IO)
- net SLA6430_74: now also IC25.8 (IO)
- net SLA6430_79: now also IC25.7 (IO)
- net SLA6430_80: now also IC25.6 (IO)
- net at CN7.1 (Pin_1): now also Q18.1 (E), R52.1
- net at CN7.3 (Pin_3): now also Q16.1 (E), R45.1
- net at CN7.5 (Pin_5): now also Q14.1 (E), R36.1
- net at CN8.1 (Pin_1): now also R3.1
- net at CN8.3 (Pin_3): now also R4.1
- net at CN8.5 (Pin_5): now also R5.1
- net at CN9.1 (Pin_1): now also R?.2
- net at IC5.10 (VccA): now also IC5.14 (VccA)
- net R_video: now reaches IC5.12 (VinA)
- net R_video: now also Q9.1 (E), R13.1
- net at IC5.13 (Vrb): now also IC6.13 (Vrb), IC7.13 (Vrb), Q8.1 (E), R7.2
- net at IC5.15 (VccD): now also IC5.9 (VccD)
- net at IC5.16 (GND): now also IC6.16 (GND), IC7.16 (GND)
- net +5VA: now reaches IC8.7 (GND)
- net +5VA: now also IC10.7 (GND), IC14.7 (GND), IC15.7 (GND), IC16.9 (GND), IC20.7 (GND), IC29.7 (GND), IC3.8 (GND), IC39.7 (GND), IC4.7 (GND), IC9.7 (GND), C1.2, C10.2, C11.2, C116.2, C12.2, C13.2, C14.2, C15,C16,C18,C20-C39,C41-C44,C47,C51,C52,C55-C57,C62-C71,C73,C75,C77,C78,C80-C89,C91-C114,C117,C118.2, C2.2, C3.2, C4.2, C45,C48,C49,C53,C60.2, C5.2, C54.2, C6.2, C61.2, C7.2, C76.2, C79.2, C8.2, C9.2, C90.2, IC22.7 (GND), IC28.8 (GND), IC36.7 (GND), IC40.7 (GND), IC44.7 (GND), IC45.7 (GND), IC46.7 (GND), Q1.2 (C), Q1.3 (B), Q13.2 (C), Q14.2 (C), Q15.2 (C), Q16.2 (C), Q17.2 (C), Q18.2 (C), Q19.2 (C), Q2.2 (C), Q2.3 (B), Q3.2 (C), Q3.3 (B), Q4.2 (C), Q5.2 (C), Q6.2 (C), Q7.2 (C), Q8.2 (C), R13.2, R15.2, R17.2, R19.2, R20.2, R21.2, R34.1, R35.2, R36.2, R37.1, R43.1, R44.2, R45.2, R46.1, R50.1, R51.2, R52.2, R53.1, R7.1, R8.1
- net at IC6.10 (VccA): now also IC6.14 (VccA)
- net G_video: now reaches IC6.12 (VinA)
- net G_video: now also Q10.1 (E), R15.1
- net at IC6.15 (VccD): now also IC6.9 (VccD)
- net at IC7.10 (VccA): now also IC7.14 (VccA)
- net B_video: now reaches IC7.12 (VinA)
- net B_video: now also Q11.1 (E), R17.1
- net at IC7.15 (VccD): now also IC7.9 (VccD)
- net SLA6170_28: now reaches IC23.28 (IO)
- net at IC26.8 (GND), IC32.15 (Eb), IC32.8 (GND)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: now also IC27.8 (GND)
- net at IC41.10 (Q3): now also R47.1
- net at IC41.12 (Q4): now also IR34.1
- net at IC41.15 (Q5): now also IR31.1
- net at IC41.2 (Q0): now also IR32.1
- net at IC41.5 (Q1): now also IR33.1
- net at IC41.7 (Q2): now also IR35.1
- net at IC31.10 (Q3): now also R40.1
- net at IC31.12 (Q4): now also IR24.1
- net at IC31.15 (Q5): now also IR21.1
- net at IC31.2 (Q0): now also IR22.1
- net at IC31.5 (Q1): now also IR23.1
- net at IC31.7 (Q2): now also IR25.1
- net at IC25.10 (Q3): now also R31.1
- net at IC25.12 (Q4): now also IR14.1
- net at IC25.15 (Q5): now also IR11.1
- net at IC25.2 (Q0): now also IR12.1
- net at IC25.5 (Q1): now also IR13.1
- net at IC25.7 (Q2): now also IR15.1
- net 15_6: no longer names the net of IC15.6, IC39.10, IC39.9, IC40.10, IC40.9, IC45.10, IC45.9, IC46.10, IC46.9
- new net: Q6.1 (E), R10.1, R16.2
- new net: Q6.3 (B), R4.2
- new net: Q12.1 (E), R19.1
- new net: Q13.1 (E), Q8.3 (B), R20.1
- new net: Q13.3 (B), R12.2, R21.1
- new net: Q4.3 (B), R12.1, R8.2
- new net: Q12.3 (B), Q4.1 (E), R6.2
- new net: Q5.1 (E), R14.2, R9.1
- new net: Q5.3 (B), R3.2
- new net: Q7.1 (E), R11.1, R18.2
- new net: Q7.3 (B), R5.2
- new net: Q10.3 (B), Q2.1 (E), R10.2
- new net: Q1.1 (E), Q9.3 (B), R9.2
- new net: Q11.3 (B), Q3.1 (E), R11.2
- new net: C76.1, Q14.3 (B), R33.1
- new net: Q15.1 (E), R33.2, R37.2
- new net: IR11.2, IR12.2, IR13.2, IR14.2, IR15.2, Q15.3 (B), R32.2, R34.2, R35.1
- new net: R31.2, R32.1
- new net: C79.1, Q16.3 (B), R42.1
- new net: Q17.1 (E), R42.2, R46.2
- new net: IR21.2, IR22.2, IR23.2, IR24.2, IR25.2, Q17.3 (B), R41.2, R43.2, R44.1
- new net: R40.2, R41.1
- new net: C90.1, Q18.3 (B), R49.1
- new net: Q19.1 (E), R49.2, R53.2
- new net: IR31.2, IR32.2, IR33.2, IR34.2, IR35.2, Q19.3 (B), R48.2, R50.2, R51.1
- new net: R47.2, R48.1
- new net 1_DA0: IC41.3 (D0), IC42.7 (Za), R?.2
- new net 1_DA1: IC41.4 (D1), IC43.9 (Zb), R?.2
- new net 1_DA2: IC33.9 (Zb), IC41.6 (D2), R?.2
- new net 1_DA3: IC33.7 (Za), IC41.11 (D3), R?.2
- new net 1_DA4: IC41.13 (D4), IC43.7 (Za), R?.2
- new net 1_DA5: IC41.14 (D5), IC42.9 (Zb), R?.2
- new net 2_DA0: IC31.3 (D0), IC32.7 (Za), R?.2
- new net 2_DA1: IC27.9 (Zb), R?.2
- new net 2_DA2: IC26.9 (Zb), IC31.6 (D2), R?.2
- new net 2_DA3: IC26.7 (Za), IC31.11 (D3), R?.2
- new net 2_DA4: IC27.7 (Za), IC31.13 (D4), R?.2
- new net 2_DA5: IC31.14 (D5), IC32.9 (Zb), R?.2
- new net 3_DA0: IC19.7 (Za), IC25.3 (D0), R?.2
- new net 3_DA1: IC18.9 (Zb), IC25.4 (D1), R?.2
- new net 3_DA2: IC17.9 (Zb), IC25.6 (D2), R?.2
- new net 3_DA3: IC17.7 (Za), IC25.11 (D3), R?.2
- new net 3_DA4: IC18.7 (Za), IC25.13 (D4), R?.2
- new net 3_DA5: IC19.9 (Zb), IC25.14 (D5), R?.2
Other:
- note added: ""1AD0""
- note added: ""1AD1""
- note added: ""1AD2""
- note added: ""1AD3""
- note added: ""1AD4""
- note added: ""1AD5""
- note added: ""2AD2""
- note added: ""2AD3""
- note added: "(ANALOG)"
- note added: "12V FAN"
- note added: "=160K"
- note added: "Connector pins (towards cartridge module) from frame unit side:\nX GND P2 P4 P6 P8 P10 P12 P14 GND\nX GND P1 P3 P5 P7 P9 P11 P13 GND\n"
- note added: "IN"
- note added: "OUT"
- note added: "Power ON led"
- note removed: ""1DA0""
- note removed: ""1DA1""
- note removed: ""1DA2""
- note removed: ""1DA3""
- note removed: ""1DA4""
- note removed: ""1DA5""
- note removed: ""2DA2""
- note removed: ""2DA3""
- moved on the sheet: 21477.2, C119, C17, C19, C50, C51, C57, C58, C59, C72, C74, CN1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

Commit message: Add files via upload
Parts:
- R99: renamed from R?; value R -> 150R
Other:
- note added: ""1DAQ0\n1DAQ1\n2DAQ0\n2DAQ1""
- note added: ""1DAQ2\n1DAQ3\n1DAQ4\n1DAQ5""
- note added: ""2DAQ2\n2DAQ3\n2DAQ4"\n2DAQ5""
- note added: ""3DAQ2\n3DAQ3\n3DAQ0\n3DAQ1""
- note added: ""3DAQ4\n3DAQ5""
- note added: "Q0...Q5 = "1DAQ0...5""
- note added: "Q0...Q5 = "2DAQ0...5""
- note added: "Q0...Q5 = "3DAQ0...5""
- note removed: ""1AD0""
- note removed: ""1AD1""
- note removed: ""1AD2""
- note removed: ""1AD3""
- note removed: ""1AD4""
- note removed: ""1AD5""
- note removed: ""2AD2""
- note removed: ""2AD3""
- note removed: ""2DA0""
- note removed: ""2DA1""
- note removed: ""2DA4""
- note removed: ""2DA5""
- note removed: ""3DA0""
- note removed: ""3DA1""
- note removed: ""3DA2""
- note removed: ""3DA3""
- note removed: ""3DA4""
- note removed: ""3DA5""
Changed lines of the file:
@@
 	14200 14250 14200 15950
 Wire Wire Line
-	11800 14250 11800 15950
-Wire Wire Line
 	24400 9800 24400 11900
 $Comp
@@
 Text GLabel 26000 12450 0    50   Input ~ 0
 5_G008_5
-Text Notes 11800 15000 0    50   ~ 0
-"1AD0"
-Text Notes 11800 15100 0    50   ~ 0
-"1AD5"
-Text Notes 11800 14800 0    50   ~ 0
-"1AD4"
-Text Notes 11800 14900 0    50   ~ 0
-"1AD1"
-Text Notes 14250 14800 0    50   ~ 0
-"1AD3"
-Text Notes 14250 14900 0    50   ~ 0
-"1AD2"
-Text Notes 14250 15000 0    50   ~ 0
-"2AD3"
-Text Notes 14250 15100 0    50   ~ 0
-"2AD2"
-Text Notes 16800 15000 0    50   ~ 0
-"2DA0"
-Text Notes 16800 15100 0    50   ~ 0
-"2DA5"
-Text Notes 16800 14800 0    50   ~ 0
-"2DA4"
-Text Notes 16800 14900 0    50   ~ 0
-"2DA1"
+Text Notes 16800 15050 0    50   ~ 0
+"2DAQ2\n2DAQ3\n2DAQ4"\n2DAQ5"
 Wire Wire Line
 	19200 15950 19950 15950
 Wire Wire Line
 	19200 14250 19200 15950
-Text Notes 19250 14800 0    50   ~ 0
-"3DA4"
-Text Notes 19250 14900 0    50   ~ 0
-"3DA1"
-Text Notes 19250 15000 0    50   ~ 0
-"3DA3"
-Text Notes 19250 15100 0    50   ~ 0
-"3DA2"
-Text Notes 25300 12400 0    50   ~ 0
-"3DA0"
-Text Notes 25300 12500 0    50   ~ 0
-"3DA5"
+Text Notes 25300 12450 0    50   ~ 0
+"3DAQ4\n3DAQ5"
 $Comp
 L 74xx:74LS54 IC46
@@
 	25150 11550 27650 11550
 $Comp
-L agg-kicad:R R?
+L agg-kicad:R R99
 U 1 1 889B4BA4
 P 25400 19300
-F 0 "R?" V 25404 19344 50  0000 L CNN
-F 1 "R" V 25495 19344 50  0000 L CNN
+F 0 "R99" V 25404 19344 50  0000 L CNN
+F 1 "150R" V 25495 19344 50  0000 L CNN
 F 2 "" H 25400 19300 50  0001 C CNN
 F 3 "" H 25400 19300 50  0001 C CNN
@@
 	1    0    0    -1
 $EndComp
+Text Notes 11800 15050 0    50   ~ 0
+"1DAQ2\n1DAQ3\n1DAQ4\n1DAQ5"
+Wire Wire Line
+	11800 14250 11800 15950
+Text Notes 14250 15050 0    50   ~ 0
+"1DAQ0\n1DAQ1\n2DAQ0\n2DAQ1"
+Text Notes 2900 12200 0    50   ~ 0
+Q0...Q5 = "3DAQ0...5"
+Text Notes 2850 14300 0    50   ~ 0
+Q0...Q5 = "2DAQ0...5"
+Text Notes 2750 16200 0    50   ~ 0
+Q0...Q5 = "1DAQ0...5"
+Text Notes 19250 15050 0    50   ~ 0
+"3DAQ2\n3DAQ3\n3DAQ0\n3DAQ1"
 $EndSCHEMATC
