File: FS-VG501/FrameUnit/analog_pcb.sch (KiCad schematic (older format))
At the start: 225 parts, among them CN201 Conn_01x7, CN4/CN206 Conn_01x10, CN5 Conn_01x10, CN7/CN205 Conn_01x06, CN8 Conn_01x06, IC201 AN5316, IC202 AN5436, IC203 4049, IC204 74LS123, IC205 7417, IC206 BA7230LS, IC207 4053, IC208 4053, IC209 4053, IC210 4053, IC211 4053, IC212 4066, IC213 4053, IC214 7406, IC215 7417, IC216 7406, IC217 4066, IC218 4066, IC219 4066, IC220 4066

Commit message: more analog circuit stuff added.
Parts:
- removed C?: 1uF/50V, symbol Device:CP
- removed Q? (x2): A564_PNP, symbol Device:Q_PNP_ECB
- removed Q?: C1684_NPN, symbol Device:Q_NPN_ECB
- removed Rx? (x2): 8K, symbol agg-kicad:R
- removed Rx?: 100K, symbol agg-kicad:R
- removed Rx?: 8K1, symbol agg-kicad:R
- removed Rx?: 4K8, symbol agg-kicad:R
- removed Rx? (x2): 4K7, symbol agg-kicad:R
- removed Rx?: 330, symbol agg-kicad:R
- added C? (x20): 1uF/50V, symbol Device:CP
- added C? (x2): 100nF, symbol agg-kicad:C
- added C?: 220pF, symbol agg-kicad:C
- added C? (x2): 1.2nF, symbol agg-kicad:C
- added C?: 33pF, symbol agg-kicad:C
- added C? (x3): 33uF/16V, symbol Device:CP
- added C?: 470uF/10V, symbol Device:CP
- added C? (x2): 5.6nF, symbol agg-kicad:C
- added L?: L, symbol agg-kicad:L
- added Q? (x16): C1684_NPN, symbol Device:Q_NPN_ECB
- added Q? (x6): A564_PNP, symbol Device:Q_PNP_ECB
- added R?: 48K, symbol agg-kicad:R
- added R? (x4), Rx? (x2): 10K, symbol agg-kicad:R
- added R?, Rx? (x6): 47K, symbol agg-kicad:R
- added R?: 36K, symbol agg-kicad:R
- added R? (x3): 1K5, symbol agg-kicad:R
- added R? (x2): 3K7, symbol agg-kicad:R
- added R?: 540, symbol agg-kicad:R
- added R?: 150, symbol agg-kicad:R
- added R?, Rx? (x6): 4K7, symbol agg-kicad:R
- added R?: 5K7, symbol agg-kicad:R
- added R?: 100, symbol agg-kicad:R
- added R?, Rx? (x2): 480, symbol agg-kicad:R
- added R?, Rx? (x15): 1K, symbol agg-kicad:R
- added R?: 3K3, symbol agg-kicad:R
- added Rx? (x2): 2K7, symbol agg-kicad:R
- added Rx? (x14): 100K, symbol agg-kicad:R
- added Rx? (x14): 8K1, symbol agg-kicad:R
- added Rx? (x6): 830, symbol agg-kicad:R
- added Rx? (x6): 1K8, symbol agg-kicad:R
- added Rx?: 460, symbol agg-kicad:R
- added Rx? (x3): 4K, symbol agg-kicad:R
- added Rx?: 220, symbol agg-kicad:R
- added Rx? (x2): 75, symbol agg-kicad:R
- added Rx? (x2): 20K, symbol agg-kicad:R
- added Rx? (x2): 730, symbol agg-kicad:R
- added Rx?: 640, symbol agg-kicad:R
- gave numbers to parts that had none: 1
- renumbered AV1_OUT to AV_OUT, AV2_OUT to MON_OUT
Connections:
- net RGB_B_IN is gone; now on net RGBIN_B: J?.20 (P20)
- net RGB_B_OUT is gone; now on net RGBTV_B: RGB_OUT.20 (P20)
- net RGB_G_IN is gone; now on net RGBIN_G: J?.19 (P19)
- net RGB_G_OUT is gone; now on net RGBTV_G: RGB_OUT.19 (P19)
- net RGB_R_IN is gone; now on net RGBIN_R: J?.15 (P15)
- net RGB_R_OUT is gone; now on net RGBTV_R: RGB_OUT.15 (P15)
- net +12V: now also Q?.1 (E), Q?.1 (E), Q?.1 (E), Q?.1 (E), Q?.1 (E), Q?.2 (C), Q?.2 (C), Q?.2 (C), Q?.2 (C), Q?.2 (C), Q?.2 (C), Q?.2 (C), Q?.2 (C), Q?.2 (C), Q?.2 (C), Rx.1, Rx?.1, Rx?.1, Rx?.1, Rx?.1, Rx?.1, Rx?.1, Rx?.1, Rx?.1, Rx?.1, Rx?.1, Rx?.1, Rx?.1, Rx?.1, Rx?.1, Rx?.1, Rx?.1, Rx?.1, Rx?.1, Rx?.1, Rx?.1, Rx?.1, Q?.1 (E), Q?.1 (E), Q?.1 (E), Q?.1 (E), Q?.1 (E), Q?.1 (E), Q?.2 (C), Q?.2 (C), Q?.2 (C), Q?.2 (C), Q?.2 (C), Q?.2 (C), Q?.2 (C), Q?.2 (C), Q?.2 (C), Q?.2 (C), Rx?.1, Rx?.1, Rx?.1, Rx?.1, Rx?.1, Rx?.1, Rx?.1, Rx?.1; no longer Q?.2 (C), Q?.2 (C), Q?.2 (C), Rx?.1, Rx?.1, Rx?.1, Rx?.1, Rx?.1, Rx?.1, Rx?.1, Rx?.1, Rx?.1
- net +5V: now also IC203.11, IC203.9, IC204.10 (B), IC204.11 (Clr), IC204.3 (Clr), Q?.2 (C), Q?.2 (C), Q?.2 (C), Rx?.1, Rx?.1, Rx?.1, Rx?.1, Rx?.1, Rx?.1, Rx?.1, Rx?.1, Rx?.1, R?.1, R?.1, R?.1, R?.2, Rx?.1, Rx?.1; no longer Q?.1 (E), Q?.1 (E), Q?.1 (E), Q?.1 (E), Q?.1 (E), Q?.2 (C), Q?.2 (C), Q?.2 (C), Q?.2 (C), Q?.2 (C), Q?.2 (C), Q?.2 (C), Q?.2 (C), Q?.2 (C), Rx.1, Rx?.1, Rx?.1, Rx?.1, Rx?.1, Rx?.1, Rx?.1, Rx?.1, Rx?.1, Rx?.1, Rx?.1, Rx?.1, Rx?.1, Rx?.1, Rx?.1, Rx?.1, Rx?.1, Rx?.1, Rx?.1, Rx?.1, Rx?.1, Rx?.1
- net CAMERA_Audio_PIN4: now also C?.2, C?.2
- net GND: now also IC204.1 (A), IC204.14 (Cext), IC204.6 (Cext), IC210.6 (Inh), IC210.7 (VEE), IC210.8 (VSS), Rx?.2, C?.1, C?.1, C?.2, C?.2, C?.2, C?.2, R?.1, R?.2, R?.2, R?.2, R?.2, R?.2, Rx?.2, Rx?.2, Rx?.2, Rx?.2, Rx?.2, Rx?.2, Rx?.2, Rx?.2, Rx?.2, Rx?.2, Rx?.2, Rx?.2, Rx?.2, Rx?.2, Rx?.2, Rx?.2, Rx?.2, Rx?.2, Rx?.2, Rx?.2, Rx?.2, Rx?.2, Rx?.2, Rx?.2, Rx?.2, Rx?.2, Rx?.2, Rx?.2, Rx?.2, Rx?.2, Rx?.2, Rx?.2, Rx?.2, Rx?.2, Rx?.2, Rx?.2, Rx?.2, Rx?.2, Rx?.2, Rx?.2, Rx?.2, Rx?.2, Rx?.2, Rx?.2, Rx?.2; no longer CN4/CN206.7 (Pin_7)
- net at IC203.2: now also IC201.18 (Blanking)
- net CNX-6: now reaches IC203.3
- net at IC203.4: now also IC204.9 (A)
- net IC202-6: now reaches IC203.5
- net IC202-6: now also R?.2
- net CNX-4: now reaches IC203.6
- net at IC203.7: now also R?.1, R?.1
- net at IC203.14: now also IC205.5
- net at IC203.15: now also IC205.3
- net at IC213.1 (Y1): now also IC210.1 (Y1), C?.2
- net RBGTV_RGB_SWITCH: now reaches IC209.11 (A), IC209.9 (C), IC211.10 (B), IC211.11 (A), IC211.9 (C), IC213.10 (B), IC213.11 (A), IC213.9 (C), IC215.8
- net RBGTV_RGB_SWITCH: now also D?.1, D?.1
- net at IC213.12 (X0): now also IC210.12 (X0), Rx?.1, Rx?.2
- net at IC213.13 (X1): now also IC210.13 (X1), Rx?.1
- net at IC213.14 (X): now also Q?.3 (B)
- net at IC213.15 (Y): now also Q?.3 (B)
- net at IC213.2 (Y0): now also IC210.2 (Y0), Rx?.1, Rx?.2
- net at IC213.4 (Z): now also IC214.9
- net at IC211.1 (Y1), Rx?.2: now also IC208.1 (Y1)
- net at C?.1, IC211.12 (X0), Rx.1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: now also IC208.12 (X0)
- net at IC211.13 (X1), Rx?.2: now also IC208.13 (X1)
- net at C?.1, IC211.2 (Y0), Rx?.1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: now also IC208.2 (Y0)
- net at C?.1, IC211.3 (Z1), Rx?.1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: now also IC208.3 (Z1)
- net at IC211.5 (Z0), Rx?.2: now also IC208.5 (Z0)
- net at IC208.10 (B), IC208.11 (A), IC208.9 (C): now also IC207.11 (A), IC209.10 (B), IC210.10 (B), IC210.11 (A), IC210.9 (C), IC215.10
- net at IC209.1 (Y1): now also IC209.3 (Z1), IC214.12
- net CN206-2: now reaches IC209.14 (X)
- net CN206-2: now also IC215.5, IC216.5
- net at IC209.15 (Y): now also IC214.1
- net at IC209.4 (Z): now also IC214.5
- net at IC210.14 (X): now also Q?.3 (B)
- net at IC210.15 (Y): now also Q?.3 (B)
- net at IC210.4 (Z): now also IC214.3
- net at IC207.2 (Y0): now also C?.1
- net SYNC2: now reaches IC212.1
- net SYNC2: now also C?.1, Rx?.1, Rx?.2
- net at IC212.6: now also IC216.2
- net YS_SWITCH: now reaches D?.2, IC212.12
- net YS_SWITCH: now also IC214.10
- net 1_SELECT: now reaches IC220.13
- net 1_SELECT: now also IC216.4, IC217.5, IC218.6
- net 2_SELECT: now reaches IC220.5
- net 2_SELECT: now also IC216.10, IC217.6, IC218.12
- net CAMERA_SELECT: now reaches IC220.6
- net CAMERA_SELECT: now also IC216.8, IC217.12, IC219.13
- net RGBTV_SELECT: now reaches IC220.12
- net RGBTV_SELECT: now also IC216.6, IC218.13, IC219.5
- net at IC219.1: now also Rx?.1, Rx?.2
- net at IC219.2: now also IC218.10, IC218.3, IC218.9, IC219.3, Q?.3 (B)
- net at IC219.4: now also Rx?.1, Rx?.2
- net 3_SELECT: now reaches IC219.12
- net 3_SELECT: now also IC216.12, IC217.13, IC218.5
- net at IC218.1: now also IC217.10, IC217.2, IC217.3, IC217.9, Q?.3 (B)
- net at IC218.2: now also Rx?.1, Rx?.2
- net at IC218.4: now also Rx?.1, Rx?.2
- net at IC218.8: now also Rx?.1, Rx?.2
- net at IC218.11: now also Rx?.1, Rx?.2
- net at IC217.1: now also Rx?.1, Rx?.2
- net at IC217.4: now also Rx?.1, Rx?.2
- net at IC217.8: now also Rx?.1, Rx?.2
- net at IC217.11: now also Rx?.1, Rx?.2
- net at IC216.1: now also Rx?.2, Rx?.2
- net CN206-3: now reaches IC216.3
- net CN206-1: now reaches IC216.9
- net CN206-4: now reaches IC216.11
- net Ys_INV: now reaches IC214.2
- net Ym_INV: now reaches IC214.4
- net Ym_INV: now also IC206.22 (HDP_IN), Rx?.2
- net CN206-9: now reaches IC214.11
- net CN206-9: now also IC214.13, IC215.13
- net CN206-8: now reaches IC215.3
- net CN206-8: now also Rx?.1
- net CN206-6_8: now reaches IC215.9
- net CN206-6: now reaches IC215.11
- net CN206-6: now also Rx?.1
- net CN206-5: now reaches IC216.13
- net at IC205.4: now also IC205.12, R?.2, R?.2
- net at IC205.6: now also IC205.10, R?.2, R?.2
- net at IC205.8: now also C?.2, Rx?.1, Rx?.2
- net CNX-8: now reaches IC205.9
- net CNX-8: now also IC205.13, R?.1
- net at IC205.11: now also R?.1, R?.2
- net at IC202.18 (VIDEOin): now also C?.1, R?.1, R?.1
- net at IC206.1 (VIDEO_OUT): now also Rx?.2
- net BA_SYNC_IN: now reaches IC206.2 (SYNC_IN)
- net BA_SYNC_IN: now also R?.1, R?.1, R?.1
- net CSVIDEO: now reaches IC206.20 (VIDEO_IN)
- net CSVIDEO: now also C?.1
- net at IC206.23 (YaP_IN): now also L?.2, Rx?.1
- net at IC204.15 (RCext): now also C?.1, R?.2
- net at IC204.5 (Q): now also R?.2
- net at IC204.7 (RCext): now also C?.2, R?.1
- net ENABLE_CS: now reaches D?.1
- net AV1_LA_OUT renamed AV_LA_OUT
- net AV_LA_OUT: now also Rx?.1
- net AV1_RA_OUT renamed AV_RA_OUT
- net AV_RA_OUT: now also Rx?.1
- net AV1_V_OUT renamed AV_V_OUT
- net AV_V_OUT: now also Rx?.1
- net AV2_LA_OUT renamed MON_LA_OUT
- net MON_LA_OUT: now also Rx?.1
- net AV2_RA_OUT renamed MON_RA_OUT
- net MON_RA_OUT: now also Rx?.1
- net AV2_V_OUT renamed MON_V_OUT
- net MON_V_OUT: now also Rx?.1
- net AV_Ctrl renamed RGBIN_AV_Ctrl
- net C-Sync_IN renamed RGBIN_C-Sync_IN
- net C-Synch_out renamed RGBTV_C-Synch_out
- net RGB_LA_in renamed RGBIN_LA_in
- net RGBIN_LA_in: now also C?.2
- net RGB_LA_out renamed RGBTV_LA_out
- net RGB_RA_in renamed RGBIN_RA_in
- net RGBIN_RA_in: now also C?.2
- net RGB_RA_out renamed RGBTV_RA_out
- net Ym_input renamed RGBIN_Ym_input
- net Ys_input renamed RGBIN_Ys_input
- new net: Q?.1 (E), Q?.3 (B), Rx?.1, Rx?.1
- new net: C?.2, Q?.1 (E), Q?.3 (B), Rx?.1
- new net: C?.1, Rx?.1 (x12)
- new net: C?.2, Q?.1 (E), Rx?.1 (x8)
- new net: Q?.2 (C), Q?.3 (B), Rx?.1 (x6)
- new net: C?.1, Rx?.1, Rx?.2 (x4)
- new net: Q?.1 (E), Rx?.1 (x6)
- new net: Q?.2 (C), Q?.3 (B), Rx?.2 (x6)
- new net: R?.1, R?.1, R?.2
- new net: C?.1, Rx?.2 (x2)
- new net: C?.1, Q?.3 (B), Rx?.1, Rx?.1
- new net: C?.2, Rx?.1, Rx?.2
- new net: C?.1, Q?.3 (B), Rx?.1, Rx?.2
- new net: C?.1, Rx?.2, Rx?.2
- new net: C?.1, Rx?.1, Rx?.2, Rx?.2 (x2)
- new net: Rx?.1, Rx?.2
- new net: L?.1, Rx?.2
- new net: C?.1, R?.1, R?.2
- new net: C?.2, R?.1
- new net: R?.1, R?.2, R?.2
- new net: C?.1, C?.2, R?.1
- new net 1_LA: C?.2
- new net 1_RA: C?.2
- new net 2_LA: C?.2
- new net 2_RA: C?.2
- new net 3_LA: C?.2
- new net 3_RA: C?.2
- new net IC201-11: C?.1, R?.2
- new net IC202-1: C?.2
- new net IC202-16: R?.2
- new net RGBIN_LA_output: Rx?.1
- new net RGBIN_RA_output: Rx?.1
- new net RGBTV_LA_OUT: Rx?.1
- new net RGBTV_LA_in: C?.2
- new net RGBTV_RA_OUT: Rx?.1
- new net RGBTV_RA_in: C?.2
- no-connect marks 2 -> 3
Other:
- note added: "B to composite \ngeneration"
- note added: "CNX"
- note added: "CNX-2"
- note added: "CNX-4"
- note added: "CNX-5"
- note added: "DIGITIZED\nRGB"
- note added: "G to composite \ngeneration"
- note added: "Left Audio Out"
- note added: "R to composite \ngeneration"
- note added: "RGB left Audio output"
- note added: "Right Audio Out"
- note added: "T1"
- note added: "Ym_signal\ninverted\nN1"
- note added: "Ys_signal\ninverted"
- note removed: "BA piiri, PIN-20"
- note removed: "IC214 = +12V"
- note removed: "IC215 = +12V"
- note removed: "IC216 = +12V"
- moved on the sheet: C?, CN4/CN206, D?, IC201, IC202, IC203A, IC203B, IC203C, IC203D, IC203E, IC203F, IC204B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

Commit message: added more analog part
Parts:
- removed Rx? (x2): 100, symbol agg-kicad:R
- removed Rx?: 75, symbol agg-kicad:R
- added J?: CAMERA_CONNECTOR, symbol agg-kicad:CONN_01x05
- added RN?: 10K, Resistor_THT:R_Array_SIP9, symbol Device:R_Network08
- added Rx? (x29): 100K, symbol agg-kicad:R
- added Rx?: 100, symbol agg-kicad:R
Connections:
- net IC201-11 is gone; now on an unnamed net: C?.1, R?.2
- net IC202-1 is gone; now on an unnamed net: C?.2
- net IC202-16 is gone; now on an unnamed net: R?.2
- net +12V: now also Rx?.1, Rx?.1, Rx?.1, Rx?.1, Rx?.1, Rx?.1, Rx?.1, Rx?.1, Rx?.1, Rx?.1, Rx?.1, Rx?.1, Rx?.1, Rx?.1, Rx?.1, Rx?.1, Rx?.1, Rx?.1, Rx?.1, Rx?.1, Rx?.1, Rx?.1, Rx?.1, Rx?.1, Rx?.1
- net 1_SELECT: now also Rx?.2
- net 2_SELECT: now also Rx?.2
- net 3_SELECT: now also Rx?.2
- net CAMERA_Audio_PIN4: now also J?.4
- net CAMERA_SELECT: now also Rx?.2
- net CN206-1: now also CN4/CN206.1 (Pin_1), RN?.2 (R1)
- net CN206-2: now also CN4/CN206.2 (Pin_2), RN?.3 (R2)
- net CN206-3: now also CN4/CN206.3 (Pin_3), RN?.4 (R3)
- net CN206-4: now also CN4/CN206.4 (Pin_4), RN?.5 (R4)
- net CN206-5: now also CN4/CN206.5 (Pin_5), RN?.6 (R5)
- net CN206-6: now also CN4/CN206.6 (Pin_6), IC203.14, IC205.5, RN?.7 (R6)
- net CN206-8: now also CN4/CN206.8 (Pin_8), RN?.8 (R7)
- net CN206-9: now also CN4/CN206.9 (Pin_9), RN?.9 (R8)
- net CN2_5: no longer CN4/CN206.6 (Pin_6)
- net CN4_1: no longer CN4/CN206.1 (Pin_1)
- net CN4_2: no longer CN4/CN206.2 (Pin_2)
- net CN4_3: no longer CN4/CN206.3 (Pin_3)
- net CN5_1: no longer CN5.1 (Pin_1)
- net CN5_3: no longer CN5.3 (Pin_3)
- net CN5_9: no longer CN5.9 (Pin_9)
- net CNX-4: now also CN5.4 (Pin_4), IC204.2 (B)
- net CNX-6: now also CN5.6 (Pin_6)
- net CNX-8: now also CN5.8 (Pin_8)
- net GND: now also CN4/CN206.7 (Pin_7), Rx?.2, Rx?.2, Rx?.2; no longer IC207.3 (Z1)
- net RBGTV_RGB_SWITCH: now also Rx?.2
- net RGBTV_SELECT: now also Rx?.2
- net SLA6170_19: no longer CN4/CN206.4 (Pin_4)
- net SLA6170_20: no longer CN4/CN206.5 (Pin_5)
- net SLA6170_22: no longer CN4/CN206.9 (Pin_9)
- net SLA6170_26: no longer CN5.4 (Pin_4)
- net SLA6170_27: no longer CN5.5 (Pin_5)
- net SLA6170_28: no longer CN5.8 (Pin_8)
- net SLA6170_30: no longer CN5.6 (Pin_6)
- net SLA6430_48: no longer CN4/CN206.8 (Pin_8)
- net YS_SWITCH: now also Rx?.2
- net at IC208.1 (Y1), IC211.1 (Y1): now also Rx?.2
- net at IC207.11 (A), IC208.10 (B), IC208.11 (A)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: now also Rx?.2
- net at IC207.13 (X1), Rx?.1, Rx?.2: no longer IC207.1 (Y1)
- net at IC207.10 (B), IC215.4: now also Rx?.2
- net at C?.1, IC207.2 (Y0): now also Rx?.1, Rx?.2
- net at IC207.5 (Z0): now also C?.1, Rx?.1, Rx?.2
- net at IC207.9 (C), IC215.12: now also Rx?.2
- net at D?.2, D?.2, IC212.13: now also Rx?.2
- net at IC212.6, IC216.2: now also Rx?.2
- net at IC219.1, Rx?.1, Rx?.2: now also Rx?.2
- net at IC219.4, Rx?.1, Rx?.2: now also Rx?.2
- net at IC218.8, Rx?.1, Rx?.2: now also Rx?.2
- net at IC218.11, Rx?.1, Rx?.2: now also Rx?.2
- net at IC217.1, Rx?.1, Rx?.2: now also Rx?.2
- net at IC217.4, Rx?.1, Rx?.2: now also Rx?.2
- net at IC217.8, Rx?.1, Rx?.2: now also Rx?.2
- net at IC217.11, Rx?.1, Rx?.2: now also Rx?.2
- net CN201-1: now reaches CN201.1 (Pin_1)
- net CN201-2: now reaches CN201.2 (Pin_2)
- net CN201-3: now reaches CN201.3 (Pin_3)
- net CN201-4: now reaches CN201.4 (Pin_4)
- net CN201-5: now reaches CN201.5 (Pin_5)
- net CN201-6: now reaches CN201.6 (Pin_6)
- net CN201-7: now reaches CN201.7 (Pin_7)
- net CNX-9: now reaches IC206.10 (BFP_IN)
- net CNX-9: now also CN5.9 (Pin_9), IC206.21 (PCP_IN)
- net CNX-3: now reaches IC204.13 (Q)
- net CNX-3: now also CN5.3 (Pin_3)
- net CNX-5: now reaches IC204.12 (~Q)
- net CNX-5: now also CN5.5 (Pin_5)
- net at IC218.2, Rx?.1, Rx?.2: now also Rx?.2
- net at C?.1, Rx?.1, Rx?.2: now also Rx?.1
- net CAMERAIN_V renamed CAMERA_V_PIN1
- net CAMERA_V_PIN1: now also J?.1
- new net: IC207.1 (Y1), Rx?.1, Rx?.2
- new net: IC207.3 (Z1), Rx?.1, Rx?.2
- new net CAMERA_12V_PIN3: J?.3
- new net CAMERA_GND_PIN2: J?.2
- new net CAMERA_GND_PIN5: J?.5
- no-connect marks 3 -> 4
Other:
- note added: "BA-pin21\n"
- note added: "CNX-3"
- note added: "IN"
- note added: "IN\n"
- note added: "Not connected"
- note added: "OUT\n"
- note removed: "CNX-2"
- moved on the sheet: C?, CN5, IC201, IC203A, IC203C, R?

Commit message: Add files via upload
Parts:
- removed unit 1 of IC205
- removed unit 1 of IC215
- removed R?: 10K, symbol agg-kicad:R
- removed Rx?: 100K, symbol agg-kicad:R
- added C?: 1uF/50V, symbol Device:CP
- added C?: 33uF/16V, symbol Device:CP
- added Q?: C1684_NPN, symbol Device:Q_NPN_ECB
- added R? (x3): 15K, symbol agg-kicad:R
- added R?: 3K3, symbol agg-kicad:R
- added R?: 4K, symbol agg-kicad:R
- added Rx?: 2K7, symbol agg-kicad:R
- added Rx? (x2): 10K, symbol agg-kicad:R
Connections:
- net 1IN_V is gone; now on net AV1_V_IN: C?.2, Rx?.1
- net 1_LA is gone; now on net AV1_LA_IN: C?.2
- net 1_RA is gone; now on net AV1_RA_IN: C?.2
- net 2IN_V is gone; now on net AV2_V_IN: C?.2, Rx?.1
- net 2_LA is gone; now on net AV2_LA_IN: C?.2
- net 2_RA is gone; now on net AV2_RA_IN: C?.2
- net 3_LA is gone; now on net AV3_LA_IN: C?.2
- net 3_RA is gone; now on net AV3_RA_IN: C?.2
- net CN201-2 is gone; now on net +12V: CN201.2 (Pin_2)
- net CN201-5 is gone; now on net GND: CN201.5 (Pin_5)
- net IC202-6 is gone; now on an unnamed net: IC203.5
- net +12V: now also IC201.12 (VCC), IC202.15 (VCC1), IC209.16 (VDD), IC211.16 (VDD), IC212.14 (VDD), IC213.16 (VDD), IC217.14 (VDD), IC218.14 (VDD), IC219.14 (VDD), IC220.14 (VDD), Q?.2 (C), R?.1, Rx?.1; no longer IC203.1 (VCC), IC204.16 (VCC)
- net +5V: now also IC203.1 (VCC), IC204.16 (VCC); no longer IC212.14 (VDD), IC217.14 (VDD), IC218.14 (VDD), IC219.14 (VDD), IC220.14 (VDD)
- net CN201-1: now also R?.1
- net GND: now also IC201.8 (GND), IC202.5 (XrayProt), IC202.9 (GND), IC206.19 (GND), R?.2, Rx?.2, Rx?.2
- net RGBTV_B: no longer RGB_OUT.20 (P20)
- net at IC208.1 (Y1), IC211.1 (Y1): now also C?.1, Rx?.1, Rx?.2; no longer Rx?.2
- net at C?.1, Rx.1, Rx.2: now also IC208.13 (X1), IC211.13 (X1); no longer IC208.12 (X0), IC211.12 (X0)
- net at C?.1, Rx?.1, Rx?.2: now also IC208.5 (Z0), IC211.5 (Z0); no longer IC208.3 (Z1), IC211.3 (Z1)
- net at IC207.1 (Y1), Rx?.1, Rx?.2: now also C?.1
- net at C?.1, IC207.5 (Z0), Rx?.1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: now also IC212.11
- net at IC220.10, IC220.2, IC220.3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: now also Q?.3 (B), Rx?.1, Rx?.2
- net at IC201.23 (PedClamp2): now also R?.1, R?.2, R?.2
- net at IC202.17 (NoiseDetIN): now also Rx?.1
- net at C?.1, IC202.18 (VIDEOin), R?.1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: now also Rx?.1
- net at IC202.2 (H_AFC_out): now also R?.1, R?.2
- net at IC202.3 (H_HoldVol): now also R?.2
- net at IC202.6 (H_OUT): now also R?.2, R?.2
- new net: IC208.12 (X0), IC211.12 (X0), Rx?.2
- new net: IC208.2 (Y0), IC211.2 (Y0), Rx?.2
- new net: IC208.3 (Z1), IC211.3 (Z1), Rx?.2
- new net: C?.1, R?.1
- new net: C?.2, Q?.1 (E), Rx?.1
- no-connect marks 4 -> 2
Other:
- note added: "RGBIN_CompositeSync\n"
- note added: "To front panel"
- note removed: "CNX-3"
- note removed: "CNX-4"
- note removed: "CNX-5"
- note removed: "U2"
- moved on the sheet: C?, CN201, CN4/CN206, IC203G, IC204C, IC206, IC212B, IC212E, IC215B, IC215F, IC216B, IC216C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

Commit message: Add files via upload
Parts:
- removed R? (x2): 10K, symbol agg-kicad:R
- removed Rx?: 37K, symbol agg-kicad:R
- removed Rx?: 273, symbol agg-kicad:R
- removed Rx?: 19K, symbol agg-kicad:R
- added C?: 100pF, symbol agg-kicad:C
- added C?: 0.47uF BP, symbol Device:C
- added C?: 0.68uF/50V, symbol Device:CP
- added C?: 2.2uF BP, symbol agg-kicad:C
- added C?: 10uF/16V, symbol Device:CP
- added C?: 10uF/16v BP, symbol agg-kicad:C
- added C?: 27pF, symbol agg-kicad:C
- added L? (x2): LTRIM, symbol Device:LTRIM
- added L? (x2): L, symbol agg-kicad:L
- added Q? (x3): C1684_NPN, symbol Device:Q_NPN_ECB
- added Q? (x2): A564_PNP, symbol Device:Q_PNP_ECB
- added R?: 273, symbol agg-kicad:R
- added R? (x2): R_Variable, symbol Device:R_Variable
- added RV?: 1K6, symbol Device:R_POT
- added Rx? (x4): 1K, symbol agg-kicad:R
- added Rx? (x2): 1K6, symbol agg-kicad:R
- added Rx?: 480, symbol agg-kicad:R
- added Rx?: 2K2, symbol agg-kicad:R
- added Rx?: 330, symbol agg-kicad:R
- added Rx?: 210, symbol agg-kicad:R
- added Rx?: 1K5, symbol agg-kicad:R
- added Rx?: 4K7, symbol agg-kicad:R
- added Rx? (x2): 10K, symbol agg-kicad:R
- added Rx?: 500, symbol agg-kicad:R
- added Rx?: 16K, symbol agg-kicad:R
- added Rx?: 100, symbol agg-kicad:R
- R?: value 47K -> 37K
Connections:
- net +12V: now also Q?.2 (C), Rx?.1, Rx?.1, Rx?.1, Rx?.1, Rx?.1
- net GND: now also C?.2, L?.2, L?.2, Q?.1 (E), Q?.2 (C), Rx?.2, Rx?.2, Rx?.2, Rx?.2, Rx?.2, Rx?.2, Rx?.2
- net R-Y-OUT: now reaches IC201.20 (R-Y)
- net R-Y-OUT: now also Rx?.1, Rx?.2
- net G-Y-OUT: now reaches IC201.21 (G-Y)
- net B-Y-OUT: now reaches IC201.22 (B-Y)
- net PICCTRL4: now reaches IC201.4 (PicCtrl4)
- net PICCTRL4: now also C?.2, L?.1, Rx?.1, Rx?.1
- net PICCTRL5: now reaches IC201.5 (PicCtrl5)
- net PICCTRL5: now also L?.2, Rx?.2
- net at IC202.16 (SyncSep_OUT), R?.2: now also R?.1
- net at IC202.17 (NoiseDetIN): now also C?.2
- net at C?.1, IC202.18 (VIDEOin), R?.1: now also R?.2, R?.2; no longer R?.1
- net at IC204.5 (Q): now also Rx?.2
- net at Q?.1 (E), Rx?.1, Rx?.2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: now also C?.1
- net at Rx?.1: now also C?.1
- net at Rx?.1: now also L?.1
- net at C?.2: now also C?.1, L?.1
- new net: C?.1, Q?.3 (B), Rx?.1, Rx?.1, Rx?.2
- new net: Q?.1 (E), Rx?.1, Rx?.1
- new net: Q?.2 (C), Q?.3 (B), Rx?.2
- new net: Q?.1 (E), Rx?.2
- new net: Q?.2 (C), Q?.3 (B), Rx?.1
- new net: C?.2, Q?.1 (E), Rx?.2
- new net: C?.1, Q?.3 (B)
- new net: Q?.1 (E), Rx?.1
- new net: C?.2, R?.1
- new net: C?.2, Q?.2 (C), Rx?.2
- new net: Q?.3 (B), Rx?.1, Rx?.1
- new net: L?.2, RV?.3
- new net: RV?.1, Rx?.1
- new net: C?.1, RV?.2
- new net GEN-H-SYNC: C?.1
Other:
- note added: "1 - from transistor\n2 -o\n3 -"
- note added: "1K\n"
- note added: "600\n"
- note added: "Qx?"
- note removed: "towards IC201"
- moved on the sheet: C?, CN201, CN5, CN8, J?, R?
