File: CANON_V30F/vram_expansion/canon_v30f_vram_expansion.sch (KiCad schematic (older format))
At the start: 6 parts, among them IC1 DRAM_4464, IC2 DRAM_4464, J1 Conn_02x12_edgeconn_vram

Commit message: Add files via upload
Parts:
- C1, C2: footprint Capacitor_THT:C_Disc_D7.5mm_W5.0mm_P7.50mm -> Capacitor_THT:C_Disc_D4.7mm_W2.5mm_P5.00mm
Changed lines of the file:
@@
 F 0 "C1" V 4704 2808 50  0000 L CNN
 F 1 "100nF" V 4795 2808 50  0000 L CNN
-F 2 "Capacitor_THT:C_Disc_D7.5mm_W5.0mm_P7.50mm" H 4700 2750 50  0001 C CNN
+F 2 "Capacitor_THT:C_Disc_D4.7mm_W2.5mm_P5.00mm" H 4700 2750 50  0001 C CNN
 F 3 "" H 4700 2750 50  0001 C CNN
 	1    4700 2750
@@
 F 0 "C2" V 4854 4308 50  0000 L CNN
 F 1 "100nF" V 4945 4308 50  0000 L CNN
-F 2 "Capacitor_THT:C_Disc_D7.5mm_W5.0mm_P7.50mm" H 4850 4250 50  0001 C CNN
+F 2 "Capacitor_THT:C_Disc_D4.7mm_W2.5mm_P5.00mm" H 4850 4250 50  0001 C CNN
 F 3 "" H 4850 4250 50  0001 C CNN
 	1    4850 4250
