File: MitsubishiGL30/keyboard_connector/mitsubishig30_keyboard_connector.kicad_pcb (KiCad board)
At the start: 2 copper layers, 37.3 x 22.5 mm, 2 parts, among them J1 MITSUBISHI GL30 KBD, J2 PHILIPS/SANYO KBD

Commit message: Add files via upload
Parts:
- J1: value MITSUBISHI GL30 KBD -> Conn_02x13_Odd_Even_mirrored
- J2: value PHILIPS/SANYO KBD -> CONN_02x13
Connections:
- J1 pad 10: Y8 -> Y9
- J1 pad 11: Y7 -> Y6
- J1 pad 12: Y6 -> Y7
- J1 pad 13: Y5 -> Y4
- J1 pad 14: Y4 -> Y5
- J1 pad 15: Y3 -> Y2
- J1 pad 16: Y2 -> Y3
- J1 pad 17: Y1 -> Y0
- J1 pad 18: Y0 -> Y1
- J1 pad 19: X7 -> X6
- J1 pad 20: X6 -> X7
- J1 pad 21: X5 -> X4
- J1 pad 22: X4 -> X5
- J1 pad 23: X3 -> X2
- J1 pad 24: X2 -> X3
- J1 pad 25: X1 -> X0
- J1 pad 26: X0 -> X1
- J1 pad 5: LEDPOWER -> KANA
- J1 pad 6: KANA -> LEDPOWER
- J1 pad 7: CAPS -> Y10
- J1 pad 8: Y10 -> CAPS
- J1 pad 9: Y9 -> Y8
Other:
- outline, holes or cut-outs redrawn
Changed lines of the file:
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@@
   (layers
     (0 F.Cu signal)
-    (31 B.Cu signal)
+    (31 B.Cu signal hide)
     (32 B.Adhes user)
     (33 F.Adhes user)
@@
       (outputformat 1)
       (mirror false)
-      (drillshape 1)
+      (drillshape 0)
       (scaleselection 1)
-      (outputdirectory ""))
+      (outputdirectory "gerber/"))
   )
   (net 0 "")
@@
     (add_net KANA)
     (add_net LEDPOWER)
+    (add_net "Net-(J2-Pad22)")
     (add_net X0)
     (add_net X1)
@@
       (effects (font (size 1 1) (thickness 0.15)))
     )
-    (fp_text value "MITSUBISHI GL30 KBD" (at -10.668 7.112) (layer F.SilkS)
+    (fp_text value Conn_02x13_Odd_Even_mirrored (at -10.668 7.112) (layer F.SilkS)
       (effects (font (size 1 1) (thickness 0.15)))
     )
     (pad 25 connect rect (at 9.36 -0.07112) (size 1 11) (layers F.Cu F.Mask)
+      (net 3 X0))
+    (pad 26 connect rect (at 9.36 -0.07366) (size 1 11) (layers B.Cu B.Mask)
       (net 2 X1))
-    (pad 26 connect rect (at 9.36 -0.07366) (size 1 11) (layers B.Cu B.Mask)
-      (net 3 X0))
     (pad 17 connect rect (at 2.24 -0.07366) (size 1 11) (layers F.Cu F.Mask)
+      (net 20 Y0))
+    (pad 19 connect rect (at 4.02 -0.07366) (size 1 11) (layers F.Cu F.Mask)
+      (net 21 X6))
+    (pad 21 connect rect (at 5.8 -0.07366) (size 1 11) (layers F.Cu F.Mask)
+      (net 22 X4))
+    (pad 23 connect rect (at 7.58 -0.07366) (size 1 11) (layers F.Cu F.Mask)
+      (net 23 X2))
+    (pad 15 connect rect (at 0.46 -0.07366) (size 1 11) (layers F.Cu F.Mask)
+      (net 19 Y2))
+    (pad 13 connect rect (at -1.32 -0.07366) (size 1 11) (layers F.Cu F.Mask)
+      (net 18 Y4))
+    (pad 11 connect rect (at -3.1 -0.07366) (size 1 11) (layers F.Cu F.Mask)
+      (net 17 Y6))
+    (pad 9 connect rect (at -4.88 -0.07366) (size 1 11) (layers F.Cu F.Mask)
+      (net 16 Y8))
+    (pad 7 connect rect (at -6.66 -0.07366) (size 1 11) (layers F.Cu F.Mask)
+      (net 15 Y10))
+    (pad 5 connect rect (at -8.44 -0.07366) (size 1 11) (layers F.Cu F.Mask)
+      (net 14 KANA))
+    (pad 3 connect rect (at -10.22 -0.07366) (size 1 11) (layers F.Cu F.Mask)
+      (net 1 GND))
+    (pad 1 connect rect (at -12 -0.07366) (size 1 11) (layers F.Cu F.Mask)
+      (net 1 GND))
+    (pad 2 connect rect (at -12 -0.07366) (size 1 11) (layers B.Cu B.Mask)
+      (net 1 GND))
+    (pad 4 connect rect (at -10.22 -0.07366) (size 1 11) (layers B.Cu B.Mask)
+      (net 1 GND))
+    (pad 6 connect rect (at -8.44 -0.07366) (size 1 11) (layers B.Cu B.Mask)
+      (net 13 LEDPOWER))
+    (pad 8 connect rect (at -6.66 -0.07366) (size 1 11) (layers B.Cu B.Mask)
+      (net 12 CAPS))
+    (pad 10 connect rect (at -4.88 -0.07366) (size 1 11) (layers B.Cu B.Mask)
+      (net 11 Y9))
+    (pad 12 connect rect (at -3.1 -0.07366) (size 1 11) (layers B.Cu B.Mask)
+      (net 10 Y7))
+    (pad 14 connect rect (at -1.32 -0.07366) (size 1 11) (layers B.Cu B.Mask)
+      (net 9 Y5))
+    (pad 16 connect rect (at 0.46 -0.07366) (size 1 11) (layers B.Cu B.Mask)
+      (net 8 Y3))
+    (pad 18 connect rect (at 2.24 -0.07366) (size 1 11) (layers B.Cu B.Mask)
       (net 4 Y1))
-    (pad 19 connect rect (at 4.02 -0.07366) (size 1 11) (layers F.Cu F.Mask)
+    (pad 20 connect rect (at 4.02 -0.07366) (size 1 11) (layers B.Cu B.Mask)
       (net 5 X7))
-    (pad 21 connect rect (at 5.8 -0.07366) (size 1 11) (layers F.Cu F.Mask)
+    (pad 22 connect rect (at 5.8 -0.07366) (size 1 11) (layers B.Cu B.Mask)
       (net 6 X5))
-    (pad 23 connect rect (at 7.58 -0.07366) (size 1 11) (layers F.Cu F.Mask)
+    (pad 24 connect rect (at 7.58 -0.07366) (size 1 11) (layers B.Cu B.Mask)
       (net 7 X3))
-    (pad 15 connect rect (at 0.46 -0.07366) (size 1 11) (layers F.Cu F.Mask)
-      (net 8 Y3))
-    (pad 13 connect rect (at -1.32 -0.07366) (size 1 11) (layers F.Cu F.Mask)
-      (net 9 Y5))
-    (pad 11 connect rect (at -3.1 -0.07366) (size 1 11) (layers F.Cu F.Mask)
-      (net 10 Y7))
-    (pad 9 connect rect (at -4.88 -0.07366) (size 1 11) (layers F.Cu F.Mask)
-      (net 11 Y9))
-    (pad 7 connect rect (at -6.66 -0.07366) (size 1 11) (layers F.Cu F.Mask)
-      (net 12 CAPS))
-    (pad 5 connect rect (at -8.44 -0.07366) (size 1 11) (layers F.Cu F.Mask)
-      (net 13 LEDPOWER))
-    (pad 3 connect rect (at -10.22 -0.07366) (size 1 11) (layers F.Cu F.Mask)
-      (net 1 GND))
-    (pad 1 connect rect (at -12 -0.07366) (size 1 11) (layers F.Cu F.Mask)
-      (net 1 GND))
-    (pad 2 connect rect (at -12 -0.07366) (size 1 11) (layers B.Cu B.Mask)
-      (net 1 GND))
-    (pad 4 connect rect (at -10.22 -0.07366) (size 1 11) (layers B.Cu B.Mask)
-      (net 1 GND))
-    (pad 6 connect rect (at -8.44 -0.07366) (size 1 11) (layers B.Cu B.Mask)
-      (net 14 KANA))
-    (pad 8 connect rect (at -6.66 -0.07366) (size 1 11) (layers B.Cu B.Mask)
-      (net 15 Y10))
-    (pad 10 connect rect (at -4.88 -0.07366) (size 1 11) (layers B.Cu B.Mask)
-      (net 16 Y8))
-    (pad 12 connect rect (at -3.1 -0.07366) (size 1 11) (layers B.Cu B.Mask)
-      (net 17 Y6))
-    (pad 14 connect rect (at -1.32 -0.07366) (size 1 11) (layers B.Cu B.Mask)
-      (net 18 Y4))
-    (pad 16 connect rect (at 0.46 -0.07366) (size 1 11) (layers B.Cu B.Mask)
-      (net 19 Y2))
-    (pad 18 connect rect (at 2.24 -0.07366) (size 1 11) (layers B.Cu B.Mask)
-      (net 20 Y0))
-    (pad 20 connect rect (at 4.02 -0.07366) (size 1 11) (layers B.Cu B.Mask)
-      (net 21 X6))
-    (pad 22 connect rect (at 5.8 -0.07366) (size 1 11) (layers B.Cu B.Mask)
-      (net 22 X4))
-    (pad 24 connect rect (at 7.58 -0.07366) (size 1 11) (layers B.Cu B.Mask)
-      (net 23 X2))
   )
   (module Connector_PinHeader_2.54mm:PinHeader_2x13_P2.54mm_Vertical (layer F.Cu)
@@
       (effects (font (size 1 1) (thickness 0.15)))
     )
-    (fp_text value "PHILIPS/SANYO KBD" (at -3.048 4.6355 180) (layer F.SilkS)
+    (fp_text value CONN_02x13 (at -3.048 4.6355 180) (layer F.SilkS)
       (effects (font (size 1 1) (thickness 0.15)))
     )
@@
   (gr_line (start 170.1165 113.7285) (end 132.842 113.7285) (layer Edge.Cuts) (width 0.05))
   (gr_line (start 170.1165 102.489) (end 170.1165 113.7285) (layer Edge.Cuts) (width 0.05))
-  (gr_line (start 162.9165 102.489) (end 170.1165 102.489) (layer Edge.Cuts) (width 0.05))
-  (gr_line (start 162.9165 91.186) (end 162.9165 102.489) (layer Edge.Cuts) (width 0.05))
-  (gr_line (start 139.2165 91.186) (end 162.9165 91.186) (layer Edge.Cuts) (width 0.05))
+  (gr_line (start 163.0735 102.489) (end 170.1165 102.489) (layer Edge.Cuts) (width 0.05))
+  (gr_line (start 163.0735 91.186) (end 163.0735 102.489) (layer Edge.Cuts) (width 0.05))
+  (gr_line (start 139.2165 91.186) (end 163.0735 91.186) (layer Edge.Cuts) (width 0.05))
   (segment (start 138.6931 103.1833) (end 139.0387 103.1833) (width 0.25) (layer F.Cu) (net 1))
   (segment (start 139.0387 103.1833) (end 139.4424 102.7796) (width 0.25) (layer F.Cu) (net 1))
