File: vhd_c9d_card/vhd_9c9.kicad_pcb (KiCad board)
At the start: 2 copper layers, 145 x 120 mm, 114 parts, among them IC1 SN751701P, IC10 8255A, IC11 27C256, IC12 4538, IC13 4030BP, IC14 4069, IC15 4013, IC16 4013, IC17 80C49C, IC18 4013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

Commit message: Add files via upload
Parts:
- added FL1: EMI_Filter_LCL, Connector_PinHeader_2.54mm:PinHeader_1x03_P2.54mm_Vertical, F.Cu at (65.4, 6.35)
- added FL2: EMI_Filter_LCL, Connector_PinHeader_2.54mm:PinHeader_1x03_P2.54mm_Vertical, F.Cu at (52.3, 16.6)
- added FL3: EMI_Filter_LCL, Connector_PinHeader_2.54mm:PinHeader_1x03_P2.54mm_Vertical, F.Cu at (56.9, 16.6)
- added FL4: EMI_Filter_LCL, Connector_PinHeader_2.54mm:PinHeader_1x03_P2.54mm_Vertical, F.Cu at (70.1, 6.35)
- added FL5: EMI_Filter_LCL, Connector_PinHeader_2.54mm:PinHeader_1x03_P2.54mm_Vertical, F.Cu at (65.4, 16.1)
- added FL6: EMI_Filter_LCL, Connector_PinHeader_2.54mm:PinHeader_1x03_P2.54mm_Vertical, F.Cu at (74.7, 6.35)
- added L2: L, Inductor_THT:L_Axial_L5.0mm_D3.6mm_P10.00mm_Horizontal_Murata_BL01RN1A2A2, F.Cu at (51.5, 6.60)
- added L3: L, Inductor_THT:L_Axial_L5.0mm_D3.6mm_P10.00mm_Horizontal_Murata_BL01RN1A2A2, F.Cu at (51.5, 11.8)
Connections:
- D1 pad 1: +5V -> (no net)
- D3 pad 2: VHD4 -> Net-(D3-Pad2)
- D4 pad 1: VHD4 -> Net-(D3-Pad2)
- J2 pad 6: (no net) -> Net-(J2-Pad6)
- J2 pad 9: (no net) -> VHD9
- Q1 pad 3: VHD4 -> Net-(D3-Pad2)
- R1 pad 2: VHD10 -> Net-(FL1-Pad3)
- R11 pad 1: VHD3 -> Net-(FL5-Pad3)
- R13 pad 2: Net-(J2-Pad7) -> VHD7
- R2 pad 1: VHD10 -> Net-(FL1-Pad3)
- R28 pad 1: (no net) -> VHD7
- R3 pad 2: VHD4 -> Net-(D3-Pad2)
- R30 pad 2: VHD9 -> Net-(R30-Pad2)
- R31 pad 1: VHD9 -> Net-(R30-Pad2)
- R5 pad 2: VHD12 -> Net-(FL3-Pad3)
- R6 pad 1: VHD12 -> Net-(FL3-Pad3)
- R7 pad 2: VHD8 -> Net-(FL4-Pad3)
- R9 pad 1: VHD8 -> Net-(FL4-Pad3)
