File: vhd_c9d_card/vhd_9c9.sch (KiCad schematic (older format))
At the start: 53 parts, among them IC1 80C49C, IC10 74LS04, IC11 SN751701P, IC12 74HC04, IC2 8255A, IC3 27C256, IC5 74LS30, IC6 74LS30, IC7 74LS27, IC8 74LS32, IC9 74LS02, J1.1 DIN41612_01x32_C, J1.2 DIN41612_01x32_A, J1.3 DIN41612_01x32_B, J2 DB9_Female, J3 DB15_Female, Q1 PNP (B641), Q2 NPN (D637), Q3 NPN (D637), Y1 6Mhz

Commit message: added c9c related circuit
added c9c related circuit for VHD6,7,9 lines, capacitor and resistor values are not known.
Parts:
- added C1, C101, C102, C103, C104, C105, C106, C110, C111, C113, C12, C13, C2, C4: 100nF, symbol agg-kicad:C
- added C10, C7, C8, C9: ?, symbol agg-kicad:C
- added C11: 100uf/6.3V, symbol Device:CP
- added D3, D4, D5, D6, D? (x2): D, symbol agg-kicad:D
- added IC13: 4069, symbol 4xxx:4069
- added IC14: 4070 (was TC4030BP), symbol 4xxx:4070
- added IC15, IC16, IC17: 4013, symbol 4xxx:4013
- added IC18: 4538, symbol 4xxx:4538
- added IC4: 80C49C, symbol MCU_Intel:8049
- added JP1-1, JP1-2, JP2-1, JP2-2, JP3-1, JP3-2, JP4: J, symbol Device:Jumper_NC_Small
- added JP5, JP6-1, JP6-2: Jumper, symbol Device:Jumper
- added L1: L, symbol agg-kicad:L
- added R10, R11, R12, R25, R5, R6: 10K, symbol agg-kicad:R
- added R14: 2K2, symbol agg-kicad:R
- added R16, R17, R18, R19, R20, R24, R25, R26: ?, symbol agg-kicad:R
- added R21: 75R ?, symbol agg-kicad:R
- added R22, R23: 220R, symbol agg-kicad:R
- added R? (x2): 4K7, symbol agg-kicad:R
- gave numbers to parts that had none: 7
Connections:
- net +5V: now also C1.1, C101.1, C102.1, C103.1, C104.1, C105.1, C106.1, C11.1, C110.1, C111.1, C113.1, C12.1, C13.1, C2.1, C4.1, D3.1, D?.1, IC13.14 (VDD), IC14.14 (VDD), IC15.14 (VDD), IC16.14 (VDD), IC17.14 (VDD), IC18.16 (VDD), IC4.40 (VCC), JP2-2.1, R10.1, R11.1, R12.1, R14.1, R16.1, R24.1, R25.1, R25.1, R26.1, R5.1, R6.1, R?.1, R?.1
- net A23: now also JP6-1.1; no longer IC11.2 (DA)
- net A24: now also JP6-2.2; no longer IC11.3 (RY)
- net B16: now also JP2-1.2
- net B18: no longer IC5.1
- net B19: now also JP1-2.1; no longer IC5.12
- net C18: now also JP3-2.2; no longer IC5.11
- net GND: now also C1.2, C101.2, C102.2, C103.2, C104.2, C105.2, C106.2, C11.2, C110.2, C111.2, C113.2, C12.2, C13.2, C2.2, C4.2, C7.2, C9.2, D4.2, D?.2, IC13.7 (VSS), IC14.12, IC14.13, IC14.2, IC14.7 (VSS), IC15.10 (R), IC15.4 (R), IC15.6 (S), IC15.7 (VSS), IC15.8 (S), IC16.10 (R), IC16.4 (R), IC16.6 (S), IC16.7 (VSS), IC16.8 (S), IC17.10 (R), IC17.4 (R), IC17.6 (S), IC17.7 (VSS), IC17.8 (S), IC18.1 (VSS), IC18.15 (VSS), IC18.8 (VSS), IC4.12 (DB.0), IC4.13 (DB.1), IC4.14 (DB.2), IC4.15 (DB.3), IC4.16 (DB.4), IC4.17 (DB.5), IC4.18 (DB.6), IC4.19 (DB.7), IC4.20 (GND), IC4.7 (EA), JP5.1, L1.1, R21.2; no longer IC1.23 (P2.2), J3.14 (P14), J3.15 (P15)
- net T0_PC5: now also R5.2
- net T1_PC7: now also R6.2
- net CLK: now reaches IC1.2 (X1), IC12.2
- net CLK: now also IC4.2 (X1), R14.2
- net RESET_: now reaches IC1.4 (~RESET~), IC12.9, R?.2
- net RESET_: now also IC4.4 (~RESET~)
- net P2.1_PC1: now reaches IC1.22 (P2.1)
- net P2.1_PC1: now also IC2.15 (PC1), JP4.1
- net P2.3_CPU2_P1.4: now reaches IC1.24 (P2.3)
- net P2.3_CPU2_P1.4: now also IC4.31 (P1.4)
- net at IC1.25 (PROG): now also R25.2
- net P1.0_CPU2_P2.0: now reaches IC1.27 (P1.0)
- net P1.0_CPU2_P2.0: now also IC4.21 (P2.0)
- net P1.1_CPU2_P2.1: now reaches IC1.28 (P1.1)
- net P1.1_CPU2_P2.1: now also IC4.22 (P2.1)
- net P1.2_CPU2_P2.2: now reaches IC1.29 (P1.2)
- net P1.2_CPU2_P2.2: now also IC4.23 (P2.2)
- net P1.3_CPU2_P2.3: now reaches IC1.30 (P1.3)
- net P1.3_CPU2_P2.3: now also IC4.24 (P2.3)
- net P1.4_CPU2_P2.4: now reaches IC1.31 (P1.4)
- net P1.4_CPU2_P2.4: now also IC4.35 (P2.4)
- net P1.5_CPU2_P2.5: now reaches IC1.32 (P1.5)
- net P1.5_CPU2_P2.5: now also IC4.36 (P2.5)
- net P1.6_CPU2_P2.6: now reaches IC1.33 (P1.6)
- net P1.6_CPU2_P2.6: now also IC4.37 (P2.6)
- net P1.7_CPU2_P2.7: now reaches IC1.34 (P1.7)
- net P1.7_CPU2_P2.7: now also IC4.38 (P2.7)
- new net: IC5.1, JP2-1.1, JP2-2.2
- new net: IC5.11, JP3-1.2, JP3-2.1
- new net: IC5.12, JP1-1.1, JP1-2.2
- new net: IC11.2 (DA), JP6-1.2
- new net: IC11.3 (RY), JP6-2.1
- new net: JP3-1.1, R10.2
- new net: J3.14 (P14), J3.15 (P15), L1.2
- new net: IC13.4, IC4.1 (T0)
- new net: IC4.25 (PROG), R12.2
- new net: IC13.12, IC4.39 (T1)
- new net: IC4.5 (~SS~), R11.2
- new net: IC15.3 (C), IC16.11 (C), IC17.1 (Q), IC17.11 (C), IC18.12 (Clk+)
- new net: IC15.11 (C), IC16.3 (C), IC17.2 (~Q), IC17.5 (D)
- new net: IC17.3 (C), IC18.5 (Clk-), IC18.7 (~Q)
- new net: D5.1, IC16.1 (Q)
- new net: IC14.4, IC16.5 (D)
- new net: D6.1, IC16.13 (Q)
- new net: IC14.10, IC16.9 (D)
- new net: IC14.6, IC15.1 (Q)
- new net: IC13.10, IC14.5, IC14.9, IC15.5 (D), IC15.9 (D), R17.2
- new net: IC14.8, IC15.13 (Q)
- new net: D?.1, D?.2, IC13.1, R22.2
- new net: D3.2, D4.1, IC13.3, R23.2
- new net: C8.1, IC13.5, R19.1, R20.2
- new net: C8.2, IC13.6, R18.1, R19.2
- new net: IC13.11, IC13.8
- new net: IC13.9, R17.1, R18.2
- new net: C7.1, IC18.2 (RxCx), R16.2
- new net: IC18.11 (Clk-), IC18.13 (R), IC18.3 (R), R26.2
- new net: C9.1, IC18.14 (RxCx), R25.2
- new net: C10.2, R20.1
- new net: D5.2, D6.2, R24.2
- new net B2: JP1-1.2
- new net CPU2_INT_: IC18.9 (~Q), IC4.6 (~INT~)
- new net CPU2_P1.6: IC4.33 (P1.6), JP4.2
- new net CPU2_P1.7: IC17.13 (Q), IC4.34 (P1.7)
- new net P2.2_CPU2_P1.5: IC1.23 (P2.2), IC4.32 (P1.5), JP5.2
- new net VHD6: C10.1, R21.1
- new net VHD7: R23.1, R?.2
- new net VHD9: R22.1, R?.2
- new net VHD9_INV: IC13.13, IC13.2, IC18.4 (Clk+)
- no-connect marks 16 -> 37
Other:
- note added: "CS1"
- note added: "JP1:\n C9D: A15 line connected (JP1-2)\n C9C: same? alternative is CS1 line (JP1-1)\nJP2\n C9D: A13 line connected (JP2-1)\n C9C: same? or alternative is +5V line (JP2-2)\nJP3:\n C9D: A14 line connected (JP3-2)\n C9C: same? or +5v line via pullup resistor (JP3-1)\nJP4: \n C9D: closed, connects 8255 PC1 to CPU2 also\n C9C: shuold be also closed\nJP5: \n C9D: closed, P2.2 input to ground\n C9C: ope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"
- note removed: "CPU2_21"
- note removed: "CPU2_22"
- note removed: "CPU2_23"
- note removed: "CPU2_24"
- note removed: "CPU2_31"
- note removed: "CPU2_33"
- note removed: "CPU2_35"
- note removed: "CPU2_36"
- note removed: "CPU2_37"
- note removed: "CPU2_38"
- moved on the sheet: D?, IC10A, IC10D, IC2E, IC3, IC8A, J1.1, J1.2, J1.3, R?

Commit message: Add files via upload
Parts:
- removed J1.1: DIN41612_01x32_C, symbol connector2:DIN41612_01x32_C
- removed J1.2: DIN41612_01x32_A, symbol connector2:DIN41612_01x32_A
- removed J1.3: DIN41612_01x32_B, symbol connector2:DIN41612_01x32_B
- removed R?: 4K7, symbol agg-kicad:R
- added J3: DIN41612_03x32_ABC, Connector_DIN:Conn_DIN41612_B096F, symbol connector2:DIN41612_03x32_ABC
- C1: renamed from C?; footprint (none) -> Capacitor_THT:C_Disc_D5.0mm_W2.5mm_P5.00mm
- C10: renamed from C12; footprint (none) -> Capacitor_THT:C_Disc_D5.0mm_W2.5mm_P5.00mm
- C11: renamed from C8; footprint (none) -> Capacitor_THT:C_Disc_D5.0mm_W2.5mm_P5.00mm
- C12: renamed from C13; footprint (none) -> Capacitor_THT:C_Disc_D5.0mm_W2.5mm_P5.00mm
- C13: renamed from C101; footprint (none) -> Capacitor_THT:C_Disc_D5.0mm_W2.5mm_P5.00mm
- C14: renamed from C9; footprint (none) -> Capacitor_THT:C_Disc_D5.0mm_W2.5mm_P5.00mm
- C15: renamed from C102; footprint (none) -> Capacitor_THT:C_Disc_D5.0mm_W2.5mm_P5.00mm
- C16: renamed from C103; footprint (none) -> Capacitor_THT:C_Disc_D5.0mm_W2.5mm_P5.00mm
- C17: renamed from C104; footprint (none) -> Capacitor_THT:C_Disc_D5.0mm_W2.5mm_P5.00mm
- C18: renamed from C105; footprint (none) -> Capacitor_THT:C_Disc_D5.0mm_W2.5mm_P5.00mm
- C19: renamed from C106; footprint (none) -> Capacitor_THT:C_Disc_D5.0mm_W2.5mm_P5.00mm
- C2: renamed from C5; footprint (none) -> Capacitor_THT:C_Disc_D5.0mm_W2.5mm_P5.00mm
- C20: renamed from C110; footprint (none) -> Capacitor_THT:C_Disc_D5.0mm_W2.5mm_P5.00mm
- C21: renamed from C111; footprint (none) -> Capacitor_THT:C_Disc_D5.0mm_W2.5mm_P5.00mm
- C22: renamed from C113; footprint (none) -> Capacitor_THT:C_Disc_D5.0mm_W2.5mm_P5.00mm
- C3: renamed from C6; footprint (none) -> Capacitor_THT:C_Disc_D5.0mm_W2.5mm_P5.00mm
- C4: renamed from C11; footprint (none) -> Capacitor_THT:CP_Radial_D10.0mm_P5.00mm
- C5: renamed from C1; footprint (none) -> Capacitor_THT:C_Disc_D5.0mm_W2.5mm_P5.00mm
- C6: renamed from C7; footprint (none) -> Capacitor_THT:C_Disc_D5.0mm_W2.5mm_P5.00mm
- C7: renamed from C2; footprint (none) -> Capacitor_THT:C_Disc_D5.0mm_W2.5mm_P5.00mm
- C8: renamed from C4; footprint (none) -> Capacitor_THT:C_Disc_D5.0mm_W2.5mm_P5.00mm
- C9: renamed from C10; footprint (none) -> Capacitor_THT:C_Disc_D5.0mm_W2.5mm_P5.00mm
- D1, D10, D13, D14, D2, D3, D4, D5, D6, D7, D8, D9: renamed from D?; footprint (none) -> Diode_THT:D_A-405_P7.62mm_Horizontal
- D11: renamed from D3; footprint (none) -> Diode_THT:D_A-405_P7.62mm_Horizontal
- D12: renamed from D4; footprint (none) -> Diode_THT:D_A-405_P7.62mm_Horizontal
- D15: renamed from D5; footprint (none) -> Diode_THT:D_A-405_P7.62mm_Horizontal
- D16: renamed from D6; footprint (none) -> Diode_THT:D_A-405_P7.62mm_Horizontal
- IC1: renamed from IC11; footprint (none) -> Package_DIP:DIP-8_W7.62mm
- IC12: renamed from IC18; footprint (none) -> Package_DIP:DIP-16_W7.62mm_Socket
- IC13, IC19: renamed from IC14; value 4070 (was TC4030BP) -> 4030BP; footprint (none) -> Package_DIP:DIP-14_W7.62mm_Socket
- IC14: renamed from IC13; footprint (none) -> Package_DIP:DIP-14_W7.62mm_Socket
- IC15: renamed from IC17; footprint (none) -> Package_DIP:DIP-16_W7.62mm_Socket
- IC15: footprint (none) -> Package_DIP:DIP-16_W7.62mm_Socket
- IC16: renamed from IC15; footprint (none) -> Package_DIP:DIP-14_W7.62mm_Socket
- IC16, IC2, IC5, IC6, IC9: footprint (none) -> Package_DIP:DIP-14_W7.62mm_Socket
- IC17: renamed from IC4; footprint (none) -> Package_DIP:DIP-40_W25.4mm_LongPads
- IC18: renamed from IC16; footprint (none) -> Package_DIP:DIP-14_W7.62mm_Socket
- IC18: renamed from IC17; footprint (none) -> Package_DIP:DIP-14_W7.62mm_Socket
- IC2: renamed from IC12; footprint (none) -> Package_DIP:DIP-14_W7.62mm_Socket
- IC3: renamed from IC10; footprint (none) -> Package_DIP:DIP-14_W7.62mm_Socket
- IC4: renamed from IC1; footprint (none) -> Package_DIP:DIP-40_W25.4mm_LongPads
- IC7: renamed from IC8; footprint (none) -> Package_DIP:DIP-14_W7.62mm_Socket
- IC8: renamed from IC7; footprint (none) -> Package_DIP:DIP-14_W7.62mm_Socket
- J1: renamed from J2; footprint (none) -> Connector_Dsub:DSUB-9_Female_Horizontal_P2.77x2.84mm_EdgePinOffset7.70mm_Housed_MountingHolesOffset9.12mm
- J2: renamed from J3; footprint (none) -> Connector_Dsub:DSUB-15_Female_Horizontal_P2.77x2.84mm_EdgePinOffset4.94mm_Housed_MountingHolesOffset7.48mm
- JP1: renamed from JP5; footprint (none) -> Connector_PinHeader_2.54mm:PinHeader_1x02_P2.54mm_Vertical
- JP1-1: renamed from JP1-2; footprint (none) -> Connector_PinHeader_2.54mm:PinHeader_1x02_P2.54mm_Vertical
- JP1-2: renamed from JP1-1; footprint (none) -> Connector_PinHeader_2.54mm:PinHeader_1x02_P2.54mm_Vertical
- JP2: renamed from JP4; footprint (none) -> Connector_PinHeader_2.54mm:PinHeader_1x02_P2.54mm_Vertical
- JP2-1: renamed from JP2-2; footprint (none) -> Connector_PinHeader_2.54mm:PinHeader_1x02_P2.54mm_Vertical
- JP2-2: renamed from JP2-1; footprint (none) -> Connector_PinHeader_2.54mm:PinHeader_1x02_P2.54mm_Vertical
- JP3-1, JP3-2, JP6-1, JP6-2: footprint (none) -> Connector_PinHeader_2.54mm:PinHeader_1x02_P2.54mm_Vertical
- L1: footprint (none) -> Inductor_THT:L_Axial_L5.0mm_D3.6mm_P10.00mm_Horizontal_Murata_BL01RN1A2A2
- Q1: renamed from Q2; footprint (none) -> Package_TO_SOT_THT:TO-92_Inline
- Q2: renamed from Q3; footprint (none) -> Package_TO_SOT_THT:TO-92_Inline
- Q3: renamed from Q1; footprint (none) -> Package_TO_SOT_THT:TO-92_Inline
- R1, R10, R11, R13, R15, R16, R19, R2, R3, R30, R5, R6, R7, R8, R9: renamed from R?; footprint (none) -> Resistor_THT:R_Axial_DIN0204_L3.6mm_D1.6mm_P7.62mm_Horizontal
- R12: renamed from R10; footprint (none) -> Resistor_THT:R_Axial_DIN0204_L3.6mm_D1.6mm_P7.62mm_Horizontal
- R14, R34: renamed from R25; footprint (none) -> Resistor_THT:R_Axial_DIN0204_L3.6mm_D1.6mm_P7.62mm_Horizontal
- R17: renamed from R7; footprint (none) -> Resistor_THT:R_Axial_DIN0204_L3.6mm_D1.6mm_P7.62mm_Horizontal
- R18: renamed from R14; footprint (none) -> Resistor_THT:R_Axial_DIN0204_L3.6mm_D1.6mm_P7.62mm_Horizontal
- R20: renamed from R3; footprint (none) -> Resistor_THT:R_Axial_DIN0204_L3.6mm_D1.6mm_P7.62mm_Horizontal
- R21: renamed from R32; footprint (none) -> Resistor_THT:R_Axial_DIN0204_L3.6mm_D1.6mm_P7.62mm_Horizontal
- R22: renamed from R002; footprint (none) -> Resistor_THT:R_Axial_DIN0204_L3.6mm_D1.6mm_P7.62mm_Horizontal
- R23: renamed from R5; footprint (none) -> Resistor_THT:R_Axial_DIN0204_L3.6mm_D1.6mm_P7.62mm_Horizontal
- R24: renamed from R6; footprint (none) -> Resistor_THT:R_Axial_DIN0204_L3.6mm_D1.6mm_P7.62mm_Horizontal
- R25: renamed from R16; footprint (none) -> Resistor_THT:R_Axial_DIN0204_L3.6mm_D1.6mm_P7.62mm_Horizontal
- R26: renamed from R21; footprint (none) -> Resistor_THT:R_Axial_DIN0204_L3.6mm_D1.6mm_P7.62mm_Horizontal
- R27: renamed from R20; footprint (none) -> Resistor_THT:R_Axial_DIN0204_L3.6mm_D1.6mm_P7.62mm_Horizontal
- R28: renamed from R23; footprint (none) -> Resistor_THT:R_Axial_DIN0204_L3.6mm_D1.6mm_P7.62mm_Horizontal
- R29: renamed from R19; footprint (none) -> Resistor_THT:R_Axial_DIN0204_L3.6mm_D1.6mm_P7.62mm_Horizontal
- R31: renamed from R22; footprint (none) -> Resistor_THT:R_Axial_DIN0204_L3.6mm_D1.6mm_P7.62mm_Horizontal
- R32: renamed from R26; footprint (none) -> Resistor_THT:R_Axial_DIN0204_L3.6mm_D1.6mm_P7.62mm_Horizontal
- R33: renamed from R18; footprint (none) -> Resistor_THT:R_Axial_DIN0204_L3.6mm_D1.6mm_P7.62mm_Horizontal
- R35: renamed from R17; footprint (none) -> Resistor_THT:R_Axial_DIN0204_L3.6mm_D1.6mm_P7.62mm_Horizontal
- R36: renamed from R12; footprint (none) -> Resistor_THT:R_Axial_DIN0204_L3.6mm_D1.6mm_P7.62mm_Horizontal
- R37: renamed from R11; footprint (none) -> Resistor_THT:R_Axial_DIN0204_L3.6mm_D1.6mm_P7.62mm_Horizontal
- R38: renamed from R24; footprint (none) -> Resistor_THT:R_Axial_DIN0204_L3.6mm_D1.6mm_P7.62mm_Horizontal
- R4: renamed from R33; footprint (none) -> Resistor_THT:R_Axial_DIN0204_L3.6mm_D1.6mm_P7.62mm_Horizontal
- Y1: footprint (none) -> Crystal:Crystal_HC18-U_Vertical
- gave numbers to parts that had none: 1
- renumbered IC2 to IC10, IC3 to IC11, IC12 to IC2
Connections:
- net A2: now also J3.A2 (Pin_a2)
- net A23: now also J3.A23 (Pin_a23)
- net A24: now also J3.A24 (Pin_a24)
- net A26: now also J3.A26 (Pin_a26)
- net A5: now also J3.A5 (Pin_a5)
- net B12: now also J3.B12 (Pin_b12)
- net B13: now also J3.B13 (Pin_b13)
- net B14: now also J3.B14 (Pin_b14)
- net B15: now also J3.B15 (Pin_b15)
- net B16: now also J3.B16 (Pin_b16)
- net B17: now also J3.B17 (Pin_b17)
- net B18: now also J3.B18 (Pin_b18)
- net B19: now also J3.B19 (Pin_b19)
- net B2: now also J3.B2 (Pin_b2)
- net B21: now also J3.B21 (Pin_b21)
- net B22: now also J3.B22 (Pin_b22)
- net B23: now also J3.B23 (Pin_b23)
- net B24: now also J3.B24 (Pin_b24)
- net B4: now also J3.B4 (Pin_b4)
- net B6: now also J3.B6 (Pin_b6)
- net B7: now also J3.B7 (Pin_b7)
- net B8: now also J3.B8 (Pin_b8)
- net C11: now also J3.C11 (Pin_c11)
- net C12: now also J3.C12 (Pin_c12)
- net C13: now also J3.C13 (Pin_c13)
- net C14: now also J3.C14 (Pin_c14)
- net C15: now also J3.C15 (Pin_c15)
- net C16: now also J3.C16 (Pin_c16)
- net C17: now also J3.C17 (Pin_c17)
- net C18: now also J3.C18 (Pin_c18)
- net C21: now also J3.C21 (Pin_c21)
- net C22: now also J3.C22 (Pin_c22)
- net C23: now also J3.C23 (Pin_c23)
- net C24: now also J3.C24 (Pin_c24)
- net C3: now also J3.C3 (Pin_c3)
- net C6: now also J3.C6 (Pin_c6)
- net C7: now also J3.C7 (Pin_c7)
- net GND: no longer IC19.12, IC19.13, IC2.11
- net at IC15.9 (D): now also D15.2, D16.2, R38.2
- new net: IC19.12, IC19.13
- new net A1: J3.A1 (Pin_a1)
- new net A10: J3.A10 (Pin_a10)
- new net A11: J3.A11 (Pin_a11)
- new net A12: J3.A12 (Pin_a12)
- new net A13: J3.A13 (Pin_a13)
- new net A14: J3.A14 (Pin_a14)
- new net A15: J3.A15 (Pin_a15)
- new net A16: J3.A16 (Pin_a16)
- new net A17: J3.A17 (Pin_a17)
- new net A18: J3.A18 (Pin_a18)
- new net A19: J3.A19 (Pin_a19)
- new net A20: J3.A20 (Pin_a20)
- new net A21: J3.A21 (Pin_a21)
- new net A22: J3.A22 (Pin_a22)
- new net A25: J3.A25 (Pin_a25)
- new net A27: J3.A27 (Pin_a27)
- new net A28: J3.A28 (Pin_a28)
- new net A29: J3.A29 (Pin_a29)
- new net A3: J3.A3 (Pin_a3)
- new net A30: J3.A30 (Pin_a30)
- new net A31: J3.A31 (Pin_a31)
- new net A32: J3.A32 (Pin_a32)
- new net A4: J3.A4 (Pin_a4)
- new net A6: J3.A6 (Pin_a6)
- new net A7: J3.A7 (Pin_a7)
- new net A8: J3.A8 (Pin_a8)
- new net A9: J3.A9 (Pin_a9)
- new net B1: J3.B1 (Pin_b1)
- new net B10: J3.B10 (Pin_b10)
- new net B11: J3.B11 (Pin_b11)
- new net B20: J3.B20 (Pin_b20)
- new net B25: J3.B25 (Pin_b25)
- new net B26: J3.B26 (Pin_b26)
- new net B27: J3.B27 (Pin_b27)
- new net B28: J3.B28 (Pin_b28)
- new net B29: J3.B29 (Pin_b29)
- new net B3: J3.B3 (Pin_b3)
- new net B30: J3.B30 (Pin_b30)
- new net B31: J3.B31 (Pin_b31)
- new net B32: J3.B32 (Pin_b32)
- new net B5: J3.B5 (Pin_b5)
- new net B9: J3.B9 (Pin_b9)
- new net C1: J3.C1 (Pin_c1)
- new net C10: J3.C10 (Pin_c10)
- new net C19: J3.C19 (Pin_c19)
- new net C2: J3.C2 (Pin_c2)
- new net C20: J3.C20 (Pin_c20)
- new net C25: J3.C25 (Pin_c25)
- new net C26: J3.C26 (Pin_c26)
- new net C27: J3.C27 (Pin_c27)
- new net C28: J3.C28 (Pin_c28)
- new net C29: J3.C29 (Pin_c29)
- new net C30: J3.C30 (Pin_c30)
- new net C31: J3.C31 (Pin_c31)
- new net C32: J3.C32 (Pin_c32)
- new net C4: J3.C4 (Pin_c4)
- new net C5: J3.C5 (Pin_c5)
- new net C8: J3.C8 (Pin_c8)
- new net C9: J3.C9 (Pin_c9)
Other:
- note added: "C9C card specific\n(empty in C9D pcb)"
- note removed: "CPU2_2"
- note removed: "VHD pins 6,7,9 \nconnected to logic\nonly in C9C pcb\n(go to 4069 ic)"
- moved on the sheet: C10, C11, C12, C13, C14, C15, C16, C17, C18, C19, C20, C21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

Commit message: Add files via upload
Parts:
- added FL1, FL2, FL3, FL4, FL5, FL6: EMI_Filter_LCL, Connector_PinHeader_2.54mm:PinHeader_1x03_P2.54mm_Vertical, symbol Device:EMI_Filter_LCL
- added L2, L3: L, Inductor_THT:L_Axial_L5.0mm_D3.6mm_P10.00mm_Horizontal_Murata_BL01RN1A2A2, symbol agg-kicad:L
Connections:
- net +5V: no longer D1.1
- net GND: now also FL1.2, FL2.2, FL3.2, FL4.2, FL5.2, FL6.2
- net VHD10: now also FL1.1; no longer R1.2, R2.1
- net VHD12: now also FL3.1; no longer R5.2, R6.1
- net VHD3: now also FL5.1; no longer R11.1
- net VHD4: now also FL2.1; no longer D3.2, D4.1, Q1.3 (C), R3.2
- net VHD6: now also L3.2
- net VHD7: now also R13.2, L2.2
- net VHD8: now also FL4.1; no longer R7.2, R9.1
- net VHD9: now also J2.9 (P9), FL6.1; no longer R30.2, R31.1
- net at J2.6: now also L3.1
- net at J2.7: now also L2.1; no longer R13.2
- new net: D3.2, D4.1, FL2.3, Q1.3 (C), R3.2
- new net: FL5.3, R11.1
- new net: FL3.3, R5.2, R6.1
- new net: FL1.3, R1.2, R2.1
- new net: FL4.3, R7.2, R9.1
- new net: R30.2, R31.1
- no-connect marks 37 -> 35
Other:
- moved on the sheet: D11, D12, D13, D14, IC14A, IC14B, R28, R30, R31

Commit message: Add files via upload
Parts:
- removed unit 2 of IC16
- removed IC17: 80C49C, Package_DIP:DIP-40_W25.4mm_LongPads, symbol MCU_Intel:8049
- removed unit 1 of IC18
- removed unit 2 of IC18
Connections:
- net +5V: now also IC4.40 (VCC)
- no-connect marks 35 -> 36
Changed lines of the file:
@@
 CLK
 $Comp
-L MCU_Intel:8049 IC17
+L MCU_Intel:8049 #IC17
 U 1 1 63585F57
 P 15000 8350
-F 0 "IC17" H 15000 10031 50  0000 C CNN
+F 0 "#IC17" H 15000 10031 50  0000 C CNN
 F 1 "80C49C" H 15000 9940 50  0000 C CNN
 F 2 "Package_DIP:DIP-40_W25.4mm_LongPads" H 15000 8550 50  0001 C CNN
@@
 $EndComp
 $Comp
-L 4xxx:4013 IC16
+L 4xxx:4013 #IC16
 U 2 1 63A8AD67
 P 14700 5400
-F 0 "IC16" H 14700 5881 50  0000 C CNN
+F 0 "#IC16" H 14700 5881 50  0000 C CNN
 F 1 "4013" H 14700 5790 50  0000 C CNN
 F 2 "Package_DIP:DIP-14_W7.62mm_Socket" H 14700 5400 50  0001 C CNN
@@
 $EndComp
 $Comp
-L 4xxx:4013 IC18
+L 4xxx:4013 #IC18
 U 2 1 63A76649
 P 16050 5900
-F 0 "IC18" H 16050 6350 50  0000 C CNN
+F 0 "#IC18" H 16050 6350 50  0000 C CNN
 F 1 "4013" H 16050 6290 50  0000 C CNN
 F 2 "Package_DIP:DIP-14_W7.62mm_Socket" H 16050 5900 50  0001 C CNN
@@
 $EndComp
 $Comp
-L 4xxx:4013 IC18
+L 4xxx:4013 #IC18
 U 1 1 63A76643
 P 16050 4850
-F 0 "IC18" H 16050 5331 50  0000 C CNN
+F 0 "#IC18" H 16050 5331 50  0000 C CNN
 F 1 "4013" H 16050 5240 50  0000 C CNN
 F 2 "Package_DIP:DIP-14_W7.62mm_Socket" H 16050 4850 50  0001 C CNN
@@
 Wire Wire Line
 	12200 8600 12200 8550
+$Comp
+L power:+5V #PWR?
+U 1 1 62E5A576
+P 5400 7950
+F 0 "#PWR?" H 5400 7800 50  0001 C CNN
+F 1 "+5V" H 5415 8123 50  0000 C CNN
+F 2 "" H 5400 7950 50  0001 C CNN
+F 3 "" H 5400 7950 50  0001 C CNN
+	1    5400 7950
+	1    0    0    -1
+$EndComp
+Wire Wire Line
+	5100 8000 5400 8000
+Wire Wire Line
+	5400 8000 5400 7950
+NoConn ~ 8800 6300
 $EndSCHEMATC
