File: rgb2scart/rgb21_scart_adapter.kicad_pcb (KiCad board)
At the start: 2 copper layers, 74.3 x 66.6 mm, 19 parts, among them J1 SCART-F, J2 RGB21, J3 DIN-8, J4 RIGHT, J5 LEFT, J6 VIDEO, U1 ICL7660

Commit message: Add files via upload
Parts:
- added C3: 220uf / 6.3V - 16V, Capacitor_THT:CP_Radial_D8.0mm_P5.00mm, F.Cu at (121.7, 141.2)
- added C4: 220uf / 6.3V - 16V, Capacitor_THT:CP_Radial_D8.0mm_P5.00mm, F.Cu at (113.0, 140.8)
- added C5: 220uf / 6.3V - 16V, Capacitor_THT:CP_Radial_D8.0mm_P5.00mm, F.Cu at (104.4, 140.4)
Connections:
- J1 pad 11: G -> G_OUT
- J1 pad 15: R -> R_OUT
- J1 pad 7: B -> B_OUT
- J3 pad 6: R -> R_OUT
- J3 pad 7: G -> G_OUT
- J3 pad 8: B -> B_OUT
Routing:
- net B_OUT: track 0.00 -> 102.2 mm
- net B: track 76.8 -> 15.7 mm, vias 1 -> 0
- net G_OUT: track 0.00 -> 52.8 mm, vias 0 -> 1
- net G: track 71.5 -> 19.7 mm, vias 2 -> 0
- net R: track 62.3 -> 20.3 mm, vias 2 -> 0
- net GND: track 250.7 -> 291.6 mm, vias 4 -> 5
- net R_OUT: track 0.00 -> 35.0 mm
- net ASPECT_RATIO: track 70.4 -> 97.2 mm
- net C_VIDEO_IN_1: track 54.0 -> 66.9 mm
- net C_VIDEO_IN: track 40.2 -> 49.4 mm
- net C_VIDEO_OUT: track 62.4 -> 53.2 mm, vias 1 -> 0
- net R_AUDIO_OUT: track 60.1 -> 68.8 mm
- net Net-(C2-Pad1): track 27.8 -> 34.2 mm
- net R_AUDIO_IN: track 48.9 -> 55.0 mm
- net RGB_switching: track 57.2 -> 52.4 mm
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Other:
- board text added: "A/V-IN 1-2=SCART 2-3=RCA"
- board text removed: "VIDEO-IN (JP5-7) 1-2 = SCART input 2-3 = RCA input"
