File: rgb2scart/rgb21_scart_adapter.sch (KiCad schematic (older format))
At the start: 19 parts, among them J1 SCART-F, J2 RGB21, J3 DIN-8, J4 RIGHT, J5 LEFT, J6 VIDEO, U1 ICL7660

Commit message: Add files via upload
Parts:
- added C3, C4, C5: 220uf / 6.3V - 16V, Capacitor_THT:CP_Radial_D8.0mm_P5.00mm, symbol Device:CP
Connections:
- net B: now also C5.1; no longer J1.7 (P7), J3.8
- net G: now also C4.1; no longer J1.11 (P11), J3.7
- net R: now also C3.1; no longer J1.15 (P15), J3.6
- new net B_OUT: C5.2, J1.7 (P7), J3.8
- new net G_OUT: C4.2, J1.11 (P11), J3.7
- new net R_OUT: C3.2, J1.15 (P15), J3.6
Changed lines of the file:
@@
 $EndComp
 Text GLabel 1700 6350 0    50   Input ~ 0
-B
+B_OUT
 Text GLabel 1700 5950 0    50   Input ~ 0
-G
+G_OUT
 Text GLabel 1700 5550 0    50   Input ~ 0
-R
+R_OUT
 Text GLabel 2900 6850 2    50   Input ~ 0
 R_AUDIO_IN_1
@@
 C_VIDEO_OUT
 Text GLabel 4250 4200 0    50   Input ~ 0
-R
+R_OUT
 Text GLabel 4850 4200 2    50   Input ~ 0
-G
+G_OUT
 Text GLabel 4550 4400 2    50   Input ~ 0
-B
+B_OUT
 $Comp
 L Regulator_SwitchedCapacitor:ICL7660 U1
@@
 SHIELD
 NoConn ~ 2900 2950
+$Comp
+L Device:CP C3
+U 1 1 62EF4385
+P 4650 5250
+F 0 "C3" H 4768 5296 50  0000 L CNN
+F 1 "220uf / 6.3V - 16V" H 4768 5205 50  0000 L CNN
+F 2 "Capacitor_THT:CP_Radial_D8.0mm_P5.00mm" H 4688 5100 50  0001 C CNN
+F 3 "~" H 4650 5250 50  0001 C CNN
+	1    4650 5250
+	1    0    0    -1
+$EndComp
+$Comp
+L Device:CP C4
+U 1 1 62EF7AD2
+P 4650 5900
+F 0 "C4" H 4768 5946 50  0000 L CNN
+F 1 "220uf / 6.3V - 16V" H 4768 5855 50  0000 L CNN
+F 2 "Capacitor_THT:CP_Radial_D8.0mm_P5.00mm" H 4688 5750 50  0001 C CNN
+F 3 "~" H 4650 5900 50  0001 C CNN
+	1    4650 5900
+	1    0    0    -1
+$EndComp
+$Comp
+L Device:CP C5
+U 1 1 62EF7F53
+P 4850 6600
+F 0 "C5" H 4968 6646 50  0000 L CNN
+F 1 "220uf / 6.3V - 16V" H 4968 6555 50  0000 L CNN
+F 2 "Capacitor_THT:CP_Radial_D8.0mm_P5.00mm" H 4888 6450 50  0001 C CNN
+F 3 "~" H 4850 6600 50  0001 C CNN
+	1    4850 6600
+	1    0    0    -1
+$EndComp
+Text GLabel 4650 5400 0    50   Input ~ 0
+R_OUT
+Text GLabel 4650 6050 0    50   Input ~ 0
+G_OUT
+Text GLabel 4850 6750 0    50   Input ~ 0
+B_OUT
+Text GLabel 4850 6450 0    50   Input ~ 0
+B
+Text GLabel 4650 5750 0    50   Input ~ 0
+G
+Text GLabel 4650 5100 0    50   Input ~ 0
+R
 $EndSCHEMATC
