File: vdh_cartridged_version_from_C9D/vhd_if_c9d.sch (KiCad schematic (older format))
At the start: 58 parts, among them IC1 80C49C, IC10 74LS04, IC12 74H004P, IC2 NEC D8255AC-2, IC3 27C256, IC6 74LS30, IC8 74LS32, IC9 74LS02, J1 Conn_02x25_Odd_Even, J3 DB15_Female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

Commit message: corrected CLK signal connection
Parts:
- added unit 6 of IC10
- added unit 2 of IC4
- added unit 3 of IC4
- added unit 1 of IC4
- renumbered IC9 to IC4
Connections:
- net CLK: now also IC12.4; no longer IC12.2, J1.42 (Pin_42)
- net GND: now also IC10.1, IC10.9, IC12.5, IC10.13, IC4.2, IC4.3, IC4.6, IC4.8; no longer IC12.11
- net at C121.1, R19.1, Y1.1: now also IC12.2, IC12.3; no longer IC12.1, IC12.6
- net at D10.1, D9.2, R11.2: now also IC12.11; no longer IC12.3
- net at IC1.6 (~INT~): now also IC12.10; no longer IC12.4
- net at C122.1, R19.2, Y1.2: now also IC12.1; no longer IC12.5
- net at IC2.6 (~CS~), IC4.11: now also IC4.4; no longer IC6.8
- new net: IC4.9, IC6.8
- new net: IC4.10, IC4.5
- no-connect marks 36 -> 47
Other:
- moved on the sheet: IC10A, IC10D, IC12G, IC6B, J1, RN2
