File: svi32x_coleco_adapter/svi_coleco_adapter.kicad_pcb (KiCad board)
At the start: 2 copper layers, 212 x 94 mm, 62 parts, among them J1 Conn_01x09, J2 Conn_01x09, J3 COLECO cartridge slot, J4 SVI external bus connector, T1 NPN_BCE_9014B, T2 NPN_BCE_9014B, U1 74LS244, U10 27C64, U11 L79L05, U2 74LS244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

Commit message: Add files via upload
Routing:
- net GND: track 0.00 -> 662.8 mm
- net +5V: track 0.00 -> 420.1 mm
- net D1: track 0.00 -> 348.3 mm
- net D2: track 0.00 -> 343.8 mm
- net D0: track 0.00 -> 342.2 mm, vias 0 -> 1
- net D3: track 0.00 -> 321.8 mm, vias 0 -> 3
- net D4: track 0.00 -> 305.8 mm, vias 0 -> 2
- net D7: track 0.00 -> 304.5 mm, vias 0 -> 2
- net D5: track 0.00 -> 294.9 mm, vias 0 -> 2
- net D6: track 0.00 -> 292.1 mm, vias 0 -> 1
- net COL_JOY8: track 0.00 -> 195.9 mm, vias 0 -> 1
- net A12: track 0.00 -> 177.2 mm
- net COL_JOY5: track 0.00 -> 169.7 mm
- net _INT: track 0.00 -> 166.9 mm, vias 0 -> 1
- net A1: track 0.00 -> 159.0 mm, vias 0 -> 1
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
Commit message: Add files via upload
Parts:
- added C30: 100nf, Capacitor_THT:C_Disc_D7.0mm_W2.5mm_P5.00mm, F.Cu at (174.6, 36.1)
- added C31: 100nf, Capacitor_THT:C_Disc_D7.0mm_W2.5mm_P5.00mm, F.Cu at (196.5, 35.9)
- added C32: 100nf, Capacitor_THT:C_Disc_D7.0mm_W2.5mm_P5.00mm, F.Cu at (209.9, 91.8)
- added C33: 100nf, Capacitor_THT:C_Disc_D7.0mm_W2.5mm_P5.00mm, F.Cu at (229.2, 91.4)
- added C34: 100nf, Capacitor_THT:C_Disc_D7.0mm_W2.5mm_P5.00mm, F.Cu at (232.7, 34.7)
- added C35: 100nf, Capacitor_THT:C_Disc_D7.0mm_W2.5mm_P5.00mm, F.Cu at (256.6, 45.8)
- added C36: 100nf, Capacitor_THT:C_Disc_D7.0mm_W2.5mm_P5.00mm, F.Cu at (252.6, 115.3)
- added C37: 100nf, Capacitor_THT:C_Disc_D7.0mm_W2.5mm_P5.00mm, F.Cu at (79.6, 91.8)
- C1, C12, C14, C15, C16, C19, C2, C21, C3, C4, C5, C6, C7, C8, C9: footprint Capacitor_THT:C_Disc_D7.5mm_W5.0mm_P7.50mm -> Capacitor_THT:C_Disc_D7.0mm_W2.5mm_P5.00mm
- C20: footprint Capacitor_THT:CP_Radial_D12.5mm_P5.00mm -> Capacitor_THT:CP_Radial_D8.0mm_P5.00mm
- R12, R14: value 22R -> 22K
- moved R9 151.3 mm to (291.5, 77.7), turned to 180 degrees
- moved R2 145.0 mm to (281.3, 74.4), turned to 0 degrees
- moved U3 144.8 mm to (237.0, 88.1), turned to 180 degrees
- moved C2 136.3 mm to (276.6, 89.2), turned to 180 degrees
- moved C6 133.2 mm to (281.5, 80.9), turned to 0 degrees
- moved R1 131.7 mm to (276.5, 76.2)
- moved R15 125.0 mm to (273.6, 84.0), turned to 180 degrees
- moved J3 121.3 mm to (181.4, 113.2)
- moved C1 119.6 mm to (276.8, 73.4), turned to 180 degrees
- moved R16 109.7 mm to (209.0, 57.7), turned to 90 degrees
- moved U7 105.8 mm to (180.7, 57.4), turned to 180 degrees
- moved C15 105.1 mm to (85.0, 61.7), turned to 90 degrees
- moved L2 104.7 mm to (70.5, 61.3)
- moved U6 103.3 mm to (202.6, 57.4), turned to 180 degrees
- moved U5 101.4 mm to (217.7, 88.4), turned to 180 degrees
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- renumbered L2 to L1, L1 to L2
Connections:
- C21 pad 1: +5V -> 5V_COL
- J3 pad 30: 5V -> 5V_COL
- L1 pad 2: +5V -> 5V_COL
Routing:
- net GND: track 662.8 -> 824.5 mm, vias 0 -> 1
- net _MREQ: track 40.4 -> 194.1 mm
- net _EXCSR: track 75.3 -> 225.4 mm
- net _CNTRL2: track 86.5 -> 221.9 mm
- net COL_JOY5: track 169.7 -> 49.6 mm
- net MINUS12V: track 82.5 -> 201.8 mm
- net _IORQ: track 25.5 -> 137.7 mm, vias 1 -> 2
- net _WR: track 26.9 -> 138.6 mm
- net J2_ENABLE: track 142.4 -> 32.3 mm
- net A15: track 23.8 -> 132.4 mm, vias 0 -> 1
- net _EXCSW: track 91.0 -> 195.3 mm, vias 2 -> 3
- net J1_ENABLE: track 147.1 -> 45.9 mm
- net _WAIT: track 59.1 -> 157.7 mm, vias 1 -> 2
- net A7: track 134.5 -> 232.4 mm, vias 2 -> 1
- net +5V: track 420.1 -> 508.2 mm
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Other:
- board size 212 x 94 mm -> 250 x 100 mm

Commit message: Add files via upload
Parts:
- added R40: 10K, Resistor_THT:R_Axial_DIN0207_L6.3mm_D2.5mm_P10.16mm_Horizontal, F.Cu at (122.0, 96.8)
- added R41: 10K, Resistor_THT:R_Axial_DIN0207_L6.3mm_D2.5mm_P10.16mm_Horizontal, F.Cu at (125.8, 105.3)
- T1, T2: value NPN_BCE_9014B -> NPN_CBE_BC547B (was 9014B)
- U10: value 27C64 -> 27C256
- moved J4 62.8 mm to (70.9, 129.0), turned to 90 degrees
- moved J3 11.4 mm to (170.1, 111.5)
- moved C12 4.02 mm to (237.2, 123.8)
- moved R3 3.91 mm to (223.8, 97.2)
- moved U11 3.86 mm to (228.2, 128.8)
- moved C11 1.71 mm to (247.8, 127.3)
- moved C20 1.44 mm to (98.5, 67.9)
Connections:
- T1 pad 1: Net-(C14-Pad2) -> Net-(R3-Pad2)
- T1 pad 2: Net-(R3-Pad2) -> Net-(C14-Pad2)
- T2 pad 1: Net-(C8-Pad2) -> Net-(R7-Pad2)
- T2 pad 2: Net-(R7-Pad2) -> Net-(C8-Pad2)
- U10 pad 1: (no net) -> Net-(R40-Pad2)
- U10 pad 14: GND -> _RAMDIS
- U10 pad 26: (no net) -> GND
- U10 pad 27: (no net) -> Net-(R41-Pad2)
Routing:
- net MINUS12V: track 201.8 -> 294.0 mm
- net _INT: track 245.7 -> 171.0 mm
- net D5: track 340.3 -> 410.9 mm, vias 3 -> 1
- net 12V: track 62.4 -> 132.2 mm
- net _WAIT: track 157.7 -> 226.2 mm, vias 2 -> 1
- net _EXCSR: track 225.4 -> 173.5 mm
- net D2: track 366.1 -> 319.8 mm, vias 1 -> 2
- net CLK: track 92.4 -> 138.4 mm, vias 1 -> 0
- net A12: track 141.9 -> 186.5 mm, vias 0 -> 1
- net _RAMDIS: track 167.6 -> 211.9 mm, vias 2 -> 1
- net A15: track 132.4 -> 176.6 mm, vias 1 -> 2
- net A1: track 202.3 -> 244.6 mm, vias 1 -> 2
- net _MREQ: track 194.1 -> 153.3 mm
- net +5V: track 508.2 -> 545.3 mm
- net GND: track 824.5 -> 859.7 mm, vias 1 -> 0
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
Commit message: Add files via upload
Parts:
- J3: footprint Connector:COLECO_30_PIN -> Connector:COLECO_30_PIN_5_02
Routing:
- net D4: track 348.6 -> 442.2 mm, vias 2 -> 0
- net D5: track 410.9 -> 342.4 mm, vias 1 -> 3
- net A14: track 188.2 -> 250.2 mm, vias 2 -> 1
- net _EXCSR: track 173.5 -> 220.2 mm, vias 2 -> 1
- net _INT: track 171.0 -> 209.4 mm, vias 0 -> 2
- net _IORQ: track 154.3 -> 117.7 mm, vias 1 -> 2
- net D6: track 333.5 -> 366.5 mm, vias 2 -> 1
- net J2_ENABLE: track 62.5 -> 29.6 mm
- net D0: track 341.6 -> 309.1 mm, vias 2 -> 3
- net A4: track 185.6 -> 159.8 mm
- net A8: track 163.7 -> 139.5 mm, vias 0 -> 1
- net A9: track 133.0 -> 157.1 mm, vias 2 -> 1
- net _EXCSW: track 211.1 -> 232.2 mm
- net _MREQ: track 153.3 -> 172.6 mm, vias 1 -> 0
- net _WR: track 132.0 -> 114.3 mm, vias 1 -> 2
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
Commit message: Add files via upload
corrected schematics, rom group pin was invalidly connected to _RAMDIS
Connections:
- U10 pad 14: _RAMDIS -> GND
Routing:
- net D5: track 342.4 -> 432.1 mm, vias 3 -> 1
- net D4: track 442.2 -> 360.2 mm, vias 0 -> 1
- net 12V: track 132.1 -> 82.7 mm
- net _CNTRL2: track 218.8 -> 267.5 mm
- net A14: track 250.2 -> 204.9 mm
- net _RAMDIS: track 202.9 -> 158.1 mm
- net _EXCSW: track 232.2 -> 195.0 mm
- net _WAIT: track 209.0 -> 179.2 mm
- net D7: track 384.3 -> 355.6 mm, vias 1 -> 2
- net _INT: track 209.4 -> 183.5 mm, vias 2 -> 0
- net A9: track 157.1 -> 134.2 mm
- net Net-(C5-Pad2): track 96.0 -> 118.6 mm
- net A8: track 139.5 -> 161.6 mm
- net A7: track 232.7 -> 254.5 mm, vias 3 -> 0
- net A5: track 197.7 -> 217.2 mm, vias 3 -> 0
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
Commit message: Add files via upload
corrected audio chip SN76489  data pin connections to datalines to reversed order, so that D0 is connected to SN76489 pin D7, D1 to pin D6, pin D2 to pin D5 and so on.
Parts:
- moved C21 1.52 mm to (207.1, 125.1)
- moved L1 1.33 mm to (192.2, 125.4)
Connections:
- U9 pad 1: D2 -> D5
- U9 pad 10: D7 -> D0
- U9 pad 11: D6 -> D1
- U9 pad 12: D5 -> D2
- U9 pad 13: D4 -> D3
- U9 pad 15: D3 -> D4
- U9 pad 2: D1 -> D6
- U9 pad 3: D0 -> D7
Routing:
- net D5: track 432.1 -> 334.3 mm, vias 1 -> 2
- net _CNTRL2: track 267.5 -> 222.6 mm
- net 12V: track 82.7 -> 125.7 mm
- net D0: track 317.0 -> 358.2 mm
- net A15: track 152.5 -> 190.0 mm, vias 2 -> 1
- net A7: track 254.5 -> 221.2 mm, vias 0 -> 3
- net _EXCSW: track 195.0 -> 226.9 mm, vias 1 -> 2
- net _WAIT: track 179.2 -> 210.8 mm
- net A1: track 215.8 -> 246.6 mm, vias 2 -> 1
- net D6: track 357.5 -> 327.9 mm
- net Net-(U3-Pad5): track 23.7 -> 52.8 mm, vias 1 -> 0
- net A4: track 159.3 -> 187.8 mm, vias 0 -> 2
- net _EXCSR: track 235.1 -> 208.2 mm, vias 1 -> 2
- net CS_A000: track 92.7 -> 70.9 mm, vias 0 -> 2
- net GND: track 875.2 -> 853.5 mm, vias 1 -> 0
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Other:
- outline, holes or cut-outs redrawn
