File: PCT-55/schematics/paxon_pct_55.sch (KiCad schematic (older format))
At the start: 455 parts, among them IC201 HA11431, IC202 TA7676AP, IC301 HA11423, IC502 _, IC901 TC4052BP, IC902 TC4052BP, IC950 HD7407, J401 CONN_01x05, J403 CONN_01x04, J404 CONN_01x07, J503 CONN_01x04, J503-1 CONN_01x04, J505 CONN_01x02, J903 CONN_01x02, J913 CONN_01x05, J918 CONN_01x02, J919 CONN_01x04, J920 CONN_01x08, J921 CONN_01x06, J927 CONN_01x03, K1 CONN_01x03, P402 CONN_01x03, P504 CONN_01x09, P801 CONN_01x03, P802 CONN_01x03, P901 CONN_01x09, P902 CONN_01x06, P903 , P911 CONN_01x05, P912 CONN_01x02, P913 CONN_01x05, P914 CONN_01x04, P917 CONN_01x02, P918 CONN_01x02, P919 CONN_01x04, P921 CONN_01x06, P927 CONN_01x03, Q203 A1015_PNP_BCE, Q204 A1015_PNP_BCE, Q301 C2073_NPN_BCE, Q302 C2073_NPN_BCE, Q303 A1015_PNP_BCE, Q304 C1815_NPN_BCE, Q351 C2610_NPN_BCE, Q352 D1425_NPN_BCE, Q451 D758_NPN_BCE, Q452 D758_NPN_BCE, Q453 D758_NPN_BCE, Q454 C1815_NPN_BCE, Q455 C1815_NPN_BCE, Q456 C1815_NPN_BCE, Q501 A1015_PNP_BCE, Q502 C1815_NPN_BCE, Q503 C2236_NPN_CBE, Q504 2SC2122A_NPN_BCE, Q505 D1052A_NPN_BCE, Q551 A733_PNP_BCE, Q801 C1815_NPN_BCE, Q802 A950_PNP_BCE, Q803 C2120_NPN_BCE, Q901 A952_PNP_BCE, Q902 C1815_NPN_BCE, Q903 A733_PNP_BCE, Q905 ???, Q906 ???, Q950 C1815_NPN_BCE, Q951 A950_PNP_BCE, Q952 C2120_NPN_BCE, Q953 C1815_NPN_BCE, Q954 C1815_NPN_BCE, Q955 C1815_NPN_BCE, SW1 CH1, SW10 MSX, SW1000 SWITCH_SPST, SW2 CH2, SW3 CH3, SW4 CH4, SW5 CH5, SW6 CH6, SW7 CH7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

Commit message: Add files via upload
Parts:
- removed P921: CONN_01x06, symbol agg-kicad:CONN_01x06
- added C201, C212, C213, C222, C227, C230, C231, C233, C234, C251, C252, C253, C254, C255, C256, C257, C258, C260, C261, C262, C290: ???, symbol agg-kicad:C
- added C203, C205, C207, C208, C263, C500: ???, symbol Device:CP1_Small
- added C206: 10nF, symbol agg-kicad:C
- added C225, C226: 10uf/25v, symbol Device:CP1_Small
- added D205: D, symbol agg-kicad:D
- added L201, L203, L207, L251, L252, L295: L, symbol agg-kicad:L
- added Q202: A854_PNP_BCE, symbol Device:Q_PNP_BCE
- added R201, R206, R207, R208, R209, R211, R212, R213, R214, R216, R217, R219, R220, R222, R225, R227, R230, R240, R244, R245, R247, R248, R249, R251, R252, R254, R255, R256, R257, R258, R259, R265, R266, R267, R268, R269, R271, R272, R280, R282, R283, R391, R523: ???, symbol agg-kicad:R
- added R526: 0R=wire, symbol agg-kicad:R
- added S201: SW_DPDT_x2, symbol Switch:SW_DPDT_x2
- added VR207, VR252, VR253, VR254, VR?: ???, symbol Device:R_POT
- added XC261: Crystal, symbol Device:Crystal
- R210: value 120R -> ???
- renumbered R277 to R242, R278 to R277, R400 to R278
Connections:
- net labels added: DARK_RED_wire_J, GREEN_wire_F, IC201_contrast_pin, IC202_pin_10, IC202_pin_2, IC202_pin_3, IC202_pin_5, IC202_pin_6, IC202_pin_9, IC301_pin_2, MINUS_15V, RED_wire_B, TP_12, TP_201, TP_31, TP_601
- net labels removed: BLUE_wire_B, YELLOW_wire_A
- wire segments 1770 -> 2093
- no-connect marks 6 -> 7
Other:
- note added: "-15V"
- note added: "<-- 64 ohm -->"
- note added: "B A -> HA11431 ContrastPin\nL L from HA11431 tonectrl\nL H msx Y video\nH L 0v\nH H from HA11431 tonectrl"
- note added: "B A -> IF-box-pin-9\nL L IF audio\nL H msx audio\nH L RCA audio in\nH H RCA audio in"
- note added: "B A CompositeVideoOut\nL L IF video\nL H 0v\nH L 0v\nH H RCA video in"
- note added: "B A SynchOut\nL L IF video\nL H msx Y video\nH L Digital RGB in synch\nH H RCA video in"
- note added: "B out\nB in"
- note added: "BP"
- note added: "G = white wire\nR\nB"
- note added: "G in\nG out"
- note added: "R in\n\nR out"
- note added: "R2x8??"
- note added: "Violet wire"
- note added: "Yellow wire A"
- note added: "audio from \nIF box"
- note added: "blue wire B"
- note added: "composite video"
- note added: "over the PCB\nwith wires"
- note added: "signal originates\nfrom MSX VDP"
- note added: "to Digital RGB PCB,\nRGB inputs level reference?"
- note added: "to front PCB"
- note added: "video from\nIF box"
- note removed: "(B) wire"
- note removed: "-15V ???"
- note removed: "B wire (red)"
- note removed: "C wire (orange)"
- note removed: "R2x8 ???"
- note removed: "R???"
- note removed: "audio from\nIF box"
- note removed: "hhhhh"
- note removed: "video from \nIF box"
- moved on the sheet: C229, C357, C378, C551, D358, IC201, J401, R229, R243, R278, R358, R423

Commit message: Add files via upload
Connections:
- net labels added: CYAN_wire_J
- net labels removed: CYAN_wire, DARK_RED_wire_J, YELLOW_wire_, wire_I
- wire segments 2093 -> 2092
Other:
- note added: "WHITE_wire_K"
- note added: "jumper wire"
- note removed: "Wire"
- moved on the sheet: C356, C358, C384
Changed lines of the file:
@@
 P 8520 14830
 F 0 "#PWR0161" H 8520 14580 50  0001 C CNN
-F 1 "GND" H 8525 14657 50  0000 C CNN
+F 1 "GND" H 8380 14750 50  0000 C CNN
 F 2 "" H 8520 14830 50  0001 C CNN
 F 3 "" H 8520 14830 50  0001 C CNN
@@
 P 8110 14830
 F 0 "#PWR0162" H 8110 14580 50  0001 C CNN
-F 1 "GND" H 8115 14657 50  0000 C CNN
+F 1 "GND" H 7950 14760 50  0000 C CNN
 F 2 "" H 8110 14830 50  0001 C CNN
 F 3 "" H 8110 14830 50  0001 C CNN
@@
 	12530 13160 12610 13160
 Connection ~ 12530 13260
-Text GLabel 8830 15180 2    50   Input ~ 0
+Text GLabel 8830 15280 2    50   Input ~ 0
 YELLOW_wire_D
 Wire Wire Line
@@
 	11550 11300 11550 11390
 Text GLabel 13940 13120 0    50   Input ~ 0
-wire_I
+GREEN_wire_I
 $Comp
 L agg-kicad:ZENER D358
@@
 $EndComp
 Text GLabel 13380 5920 0    50   Input ~ 0
-YELLOW_wire_
+YELLOW_wire_D
 Wire Wire Line
 	11070 14910 11070 15030
@@
 	12530 6250 12530 6200
 Wire Wire Line
-	12530 6200 12750 6200
-Wire Wire Line
 	12530 6180 12530 6200
 Connection ~ 12530 6200
@@
 	12530 6200 12530 6090
 Text GLabel 12530 6090 0    50   Input ~ 0
-CYAN_wire
+CYAN_wire_J
 Wire Wire Line
 	14270 6010 14270 5600
@@
 	7490 14180 7050 14180
 Wire Wire Line
-	8720 15180 8830 15180
-Connection ~ 8580 15180
+	8720 15280 8830 15280
+Connection ~ 8580 15280
 Wire Wire Line
-	8580 15180 8580 15190
+	8580 15280 8580 15290
 Wire Wire Line
-	8620 15180 8580 15180
+	8620 15280 8580 15280
 $Comp
 L agg-kicad:C C384
 U 1 1 6ED58BC8
-P 8620 15180
-F 0 "C384" H 8670 15250 50  0000 C CNN
-F 1 "10nF" H 8670 15100 50  0000 C CNN
-F 2 "" H 8620 15180 50  0001 C CNN
-F 3 "" H 8620 15180 50  0001 C CNN
-	1    8620 15180
+P 8620 15280
+F 0 "C384" H 8670 15350 50  0000 C CNN
+F 1 "10nF" H 8670 15200 50  0000 C CNN
+F 2 "" H 8620 15280 50  0001 C CNN
+F 3 "" H 8620 15280 50  0001 C CNN
+	1    8620 15280
 	1    0    0    -1
 $EndComp
-Connection ~ 8310 15180
+Connection ~ 8310 15280
 Wire Wire Line
-	8310 15180 8580 15180
+	8310 15280 8580 15280
 Wire Wire Line
-	8310 15180 8310 15220
+	8310 15280 8310 15320
 Wire Wire Line
-	8200 15180 8310 15180
+	8200 15280 8310 15280
 $Comp
 L power:GND #PWR0171
 U 1 1 6E9FC3F2
-P 8310 15450
-F 0 "#PWR0171" H 8310 15200 50  0001 C CNN
-F 1 "GND" H 8315 15277 50  0000 C CNN
-F 2 "" H 8310 15450 50  0001 C CNN
-F 3 "" H 8310 15450 50  0001 C CNN
-	1    8310 15450
+P 8310 15550
+F 0 "#PWR0171" H 8310 15300 50  0001 C CNN
+F 1 "GND" H 8160 15480 50  0000 C CNN
+F 2 "" H 8310 15550 50  0001 C CNN
+F 3 "" H 8310 15550 50  0001 C CNN
+	1    8310 15550
 	1    0    0    -1
 $EndComp
 Wire Wire Line
-	8310 15450 8310 15320
+	8310 15550 8310 15420
 $Comp
 L agg-kicad:C C358
 U 1 1 6E9FC3EB
-P 8310 15220
-F 0 "C358" V 8320 15380 50  0000 C CNN
-F 1 "18nF" V 8410 15380 50  0000 C CNN
-F 2 "" H 8310 15220 50  0001 C CNN
-F 3 "" H 8310 15220 50  0001 C CNN
-	1    8310 15220
+P 8310 15320
+F 0 "C358" V 8320 15480 50  0000 C CNN
+F 1 "18nF" V 8410 15480 50  0000 C CNN
+F 2 "" H 8310 15320 50  0001 C CNN
+F 3 "" H 8310 15320 50  0001 C CNN
+	1    8310 15320
 	0    1    1    0
 $EndComp
@@
 L agg-kicad:C C356
 U 1 1 6E9227E7
-P 8100 15180
-F 0 "C356" H 8150 15250 50  0000 C CNN
-F 1 "39nF" H 8150 15100 50  0000 C CNN
-F 2 "" H 8100 15180 50  0001 C CNN
-F 3 "" H 8100 15180 50  0001 C CNN
-	1    8100 15180
+P 8100 15280
+F 0 "C356" H 8150 15350 50  0000 C CNN
+F 1 "39nF" H 8150 15200 50  0000 C CNN
+F 2 "" H 8100 15280 50  0001 C CNN
+F 3 "" H 8100 15280 50  0001 C CNN
+	1    8100 15280
 	1    0    0    -1
 $EndComp
@@
 	7050 14460 7840 14460
 Wire Wire Line
-	7840 14460 7840 15180
-Wire Wire Line
-	7840 15180 8100 15180
+	7840 15280 8100 15280
 Wire Wire Line
 	9140 14030 9130 14030
@@
 	0    1    -1   0
 $EndComp
-Text Notes 12620 10870 0    59   ~ 0
+Text Notes 12660 10810 0    59   ~ 0
 (VVV)\nwires
 $Comp
@@
 Wire Wire Line
 	13410 11280 13460 11280
-Text Notes 13250 11240 0    59   ~ 0
-Wire
+Text Notes 13160 11210 0    59   ~ 0
+jumper wire
 $Comp
 L agg-kicad:CONN_01x02 P912
@@
 Wire Wire Line
 	16350 13330 16390 13330
-Text Notes 12650 10610 0    59   ~ 0
+Text Notes 12690 10600 0    59   ~ 0
 MSX
-Text Notes 12910 10520 0    59   ~ 0
+Text Notes 12900 10930 0    59   ~ 0
 audio
-Text Notes 12930 10860 0    59   ~ 0
+Text Notes 12930 10830 0    59   ~ 0
 R-Y
 Text Notes 12930 10720 0    59   ~ 0
 B-Y
-Text Notes 13030 10970 0    59   ~ 0
+Text Notes 13060 10520 0    59   ~ 0
 Y
 Text Notes 11320 9960 0    59   ~ 0
@@
 Wire Wire Line
 	12210 9960 13020 9960
-Text Notes 12300 9970 0    50   ~ 0
-white wire
+Text Notes 12300 9950 0    50   ~ 0
+WHITE_wire_K
 $Comp
 L agg-kicad:R R523
@@
 	21800 7680 21800 8510
 Text GLabel 21710 8910 2    50   Input ~ 0
-DARK_RED_wire_J
+CYAN_wire_J
 Wire Wire Line
 	22320 8750 22460 8750
@@
 Wire Wire Line
 	22460 8750 22490 8750
-Text GLabel 12660 5960 0    50   Input ~ 0
-DARK_RED_wire_J
-Wire Wire Line
-	12660 5960 12750 5960
-Wire Wire Line
-	12750 5960 12750 6200
-Connection ~ 12750 6200
-Wire Wire Line
-	12750 6200 12810 6200
 Wire Wire Line
 	14270 6110 14020 6110
@@
 Text Notes 14490 6470 0    50   ~ 0
 to front PCB
+Wire Wire Line
+	12530 6200 12810 6200
+Text GLabel 8370 15060 2    50   Input ~ 0
+RED_wire_E
+Wire Wire Line
+	7840 14460 7840 15280
+Wire Wire Line
+	8310 15280 8310 15060
+Wire Wire Line
+	8310 15060 8370 15060
+Text Notes 15430 11580 0    59   ~ 0
+(LLL) wires
 $EndSCHEMATC

Commit message: Add files via upload
Parts:
- removed C231, C233, C234, C257, C262: ???, symbol agg-kicad:C
- removed R225: 22R, symbol agg-kicad:R
- removed R227: 2K2, symbol agg-kicad:R
- removed R230: ???, symbol agg-kicad:R
- removed R460, R467, R468: R, symbol agg-kicad:R
- removed VR207: ???, symbol Device:R_POT
- added C231, C233, C234: 0.47uf/50v, symbol Device:CP1_Small
- added C257: 0.47uf/25v, symbol Device:CP1_Small
- added C262: 2.2uf/50v, symbol Device:CP1_Small
- added C270, C519, C564: 10nF, symbol agg-kicad:C
- added C304: 6.8nF, symbol agg-kicad:C
- added C508: 2.2nF, symbol agg-kicad:C
- added R589: 5K6, symbol agg-kicad:R
- C1000: value 22pF -> 82pF
- C201, C251: value ??? -> 56pF
- C203: value ??? -> 47uf/25v
- C205: value ??? -> 100uf/16v
- C207, C208: value ??? -> 10uf/25v
- C212, C213: value ??? -> 2.2nF
- C222, C253, C254: value ??? -> 100pF
- C227: value ??? -> 4.7uf/25v BP
- C230, C255, C256: value ??? -> 10nF
- C252: value ??? -> 33pF
- C258: value ??? -> 39pF
- C260: value ??? -> 27pF
- C261: value ??? -> 33nF
- C263: value ??? -> 1uf/50v
- C290: value ??? -> 82pF
- C500: value ??? -> 4.7uf/50v
- L201: value L -> 3 mH
- L207: value L -> 0 µH
- L251, L252: value L -> 50 µH
- L505, L506: value L -> 330uH
- L950: value L -> 700 µH
- R201, R251: value ??? -> 560R
- R206, R252, R268, R282: value ??? -> 1K
- R207, R256: value ??? -> 2K7
- R208: value ??? -> 3K3
- R209: value ??? -> 100R
- R210: value ??? -> 120R
- R211: value ??? -> 10R
- R212, R227, R258, R259: value ??? -> 2K2
- R213, R244, R245, R247: value ??? -> 470R
- R214, R240: value ??? -> 3K9
- R216: value ??? -> 0R = wire
- R217: value ??? -> 660R
- R219, R220: value ??? -> 680R
- R222: value ??? -> 150K
- R225, R266, R283: value ??? -> 10K
- R238: renamed from R278; value 1K8 -> 1K5
- R243: value 1K5 -> 1K8
- R248: value ??? -> 12K
- R249: value ??? -> 56K
- R254: value ??? -> 220R
- R255: value ??? -> 1K2
- R257: value ??? -> 220K
- R265: value ??? -> 470K
- R267: value ??? -> 1K8
- R269: value ??? -> 8K2
- R271: value ??? -> 17K
- R272: value ??? -> 16K
- R280, R523: value ??? -> 4K7
- R356: renamed from R256; value 2K7 -> 5K6
- R391: value ??? -> 1M
- gave numbers to parts that had none: 1
Connections:
- net labels added: IC202_B_DATA_IN, IC202_B_OUT, IC202_ColorContrast, IC202_FieldBlanking, IC202_G_DATA_IN, IC202_G_OUT, IC202_LineClampPulse, IC202_R_DATA_IN, IC202_R_OUT, IC202_brightness, IC301_VB_Sharp
- net labels removed: IC202_pin_10, IC202_pin_13, IC202_pin_14, IC202_pin_16, IC202_pin_17, IC202_pin_2, IC202_pin_3, IC202_pin_5, IC202_pin_6, IC202_pin_9, IC301_pin_17
- wire segments 2092 -> 2097
Other:
- note added: "-->"
- note added: "<--"
- note added: "L207 coil color code:\nBlack-Black-Brown-Gold"
- note added: "SecamSel (MSX or composite/RF)"
- note added: "VideoDataSel"
- note added: "VideoDataSel\nto IC202 (TA7676AP)"
- note added: "near JM10"
- note added: "or 2K0"
- note removed: "B out\nB in"
- note removed: "BP"
- note removed: "G in\nG out"
- note removed: "R in\n\nR out"
- note removed: "R2x8??"
- moved on the sheet: C255, C265, D205, J505, R238, R243, R258, R391, R463, R464, R465

Commit message: Add files via upload
Parts:
- C261: value 33nF -> 33nF Paper
- C302, C307: value 22nF -> 22nF Paper
- C306: value 2.2uf/16v -> 2.2uf/16v Tantal
- C355: value 6.8nF -> 6.8nF Paper
- C357: value 1.1nF -> 1.1nF Paper
- C358: value 18nF -> 18nF Paper
- C384: value 10nF -> 10nF Paper
- C901: value 82nF -> 82nF Paper
- L203: value L -> ???
- L205: renamed from L295; value L -> 50uH
- L351: value L -> 15mH
- L388: value L -> 00257
- L389: value L -> 4.7mH
- P903: value (none) -> CONN_01x02
Connections:
- net labels added: ORANGE_wire_C_RGBAmplitude, RED_wire_B_SelectAB
- net labels removed: J927_pin_3, ORANGE_wire_C, RED_wire_B
- wire segments 2097 -> 2101
Other:
- note added: "(CCC) wires,\nto Digital RGB input pcb ->J503"
- note added: "--->"
- note added: "<-"
- note added: "<-- Power to \nRGB input IC"
- note added: "<-blue wire->"
- note added: "RefVoltage\nR\nG\nB"
- note added: "SelB SelA --> selected input\n---------------------\nL L RF channel\nL H MSX\nH L Digital RGB\nH H RCA"
- note added: "SelectA and\nSecamSel (MSX or composite/RF)"
- note added: "SelectB"
- note added: "Set both\nSelectA and B"
- note added: "TUNER_15V"
- note added: "VideoDataSel -->"
- note added: "VideoDataSelOutput"
- note added: "hold memory"
- note added: "hold memory -->"
- note added: "to AFC_FB -->"
- note added: "to Digital RGB PCB,\nRGB input conversion applitude?"
- note added: "when VideoDataSel=15v, \nthat goes as power to \ndigital RGB input ic also"
- note added: "wire with magnet\ncoated around it"
- note removed: "(CCC) wires"
- note removed: "SecamSel (MSX or composite/RF)"
- note removed: "VideoDataSel"
- note removed: "to Digital RGB PCB,\nRGB inputs level reference?"
- moved on the sheet: IC950D, IC950G, L203, P927, R986

Commit message: Add files via upload
Parts:
- added C501: C, symbol agg-kicad:C
- added L501: _, symbol Device:Transformer_1P_1S
- added L? (x6): L, symbol agg-kicad:L
- added T353: FLYBACK_TRANSFORMER, symbol Video:FLYBACK_TRANSFORMER
- added TH501: 5R0M (M) 48, symbol Device:Thermistor
- S501: renamed from SW1000; value SWITCH_SPST -> Power_Switch
- renumbered F1 to F501
Connections:
- net labels added: DEGAUS_WIRE_1, DEGAUS_WIRE_2, FLYBACK_pin_6
- net labels removed: H_pin_1, H_pin_2, H_pin_3, K_pin_1, K_pin_2, K_pin_3
- wire segments 2101 -> 2149
Other:
- note added: "120V ???"
- note added: "BLUE COLOR"
- note added: "FLYBACK pin-3"
- note added: "FLYBACK pin-5"
- note added: "FLYBACK transformer\nfrom solder side"
- note added: "Fat RED wire (not the big red wire for anode)\nfrom flyback transformer"
- note added: "GREEN COLOR"
- note added: "G\nR\nB"
- note added: "NOTE!"
- note added: "PINS 1, 2/8, 4,5 and 9 are connected together someway"
- note added: "PINS 3,5,10 are connected together someway"
- note added: "RED COLOR"
- note added: "Separate black thick ground wires towards:\n-tube ground\n-tuner box metal\n-digital RGB board\n\nThere is also thick black wire from \ndigital RGB pcb to tuner box metal"
- note removed: "Fat RED wire \nfrom flyback transformer"
- note removed: "green\nwire"
- moved on the sheet: C458, F501, S501

Commit message: Add files via upload
Parts:
- XC261: value Crystal -> 3.579545Mhz
Changed lines of the file:
@@
 P 20100 14710
 F 0 "XC261" H 20120 14540 50  0000 C CNN
-F 1 "Crystal" H 20110 14460 50  0000 C CNN
+F 1 "3.579545Mhz" H 20110 14460 50  0000 C CNN
 F 2 "" H 20100 14710 50  0001 C CNN
 F 3 "~" H 20100 14710 50  0001 C CNN

Commit message: Add files via upload
Parts:
- removed L? (x6): L, symbol agg-kicad:L
- C378: value 56nF -> 56nF/200v
- L352, L353, L504: value L -> ferrite bead
- renumbered R2001 to R355, R2002 to R363
Connections:
- wire segments 2149 -> 2158
- no-connect marks 7 -> 8
Other:
- note added: "( S )"
- note added: "( W )"
- note added: "From flyback transformer, there comes also\n-big red wire (to tube Anode)\n-thick red wire (to tube neck pcb), \n to tube pin 8 ( >100V)\n-thick black wire (to tube neck pcb), \n into white plastic case,\n goes to tube pin 1/2 (Focus/kV )?\n"
- note added: "Horizontal\nAmplitude\n(wire set to S )"
- note added: "R363 pin loose --|"
- note added: "When measuring resistance between transformer pins:\n-1,2 have about zero ohms between themselfs\n-3,4,5 have about zero ohms between themselfs\n-6,7,8,9,10,11 have about zero ohms between themselfs\n-9,10,11 are connected to ground\n-3,5,10 have about zero ohms between themselfs"
- note added: "When measuring resistance between transformer pins:\n-1,2,4,5,8,9 have about zero ohms between themselfs\n-3,5,10 have about zero ohms between themselfs"
- note added: "wire-->"
- note removed: "PINS 1, 2/8, 4,5 and 9 are connected together someway"
- note removed: "PINS 3,5,10 are connected together someway"
- note removed: "wire with magnet\ncoated around it"
- moved on the sheet: C365, C378, C389, L388, L389, R389, R4000
