File: PCT-55/schematics/msx_pcb.sch (KiCad schematic (older format))
At the start: 57 parts, among them IC1 74LS157, IC10 74LS157, IC11 8255, IC12 74LS153, IC13 74LS156, IC14 74LS145, IC15 TMS9928ANL, IC16 DRAM_8118, IC17 DRAM_8118, IC18 DRAM_8118, IC19 DRAM_8118, IC2 DRAM_4416, IC20 DRAM_8118, IC21 DRAM_8118, IC22 DRAM_8118, IC23 DRAM_8118, IC24 74LS374, IC25 74HC14, IC26 74LS32, IC27 HD61J209F0, IC28 DRAM_4416, IC29 DRAM_4416, IC3 74LS157, IC4 DRAM_4416, IC5 27C128, IC6 Z80CPU, IC7 PSG_AY-3-8910, IC8 HD7417, IC9 74LS157, J1 DB9_Male, J2 DB9_Male

Commit message: more MSX pcb schematics
Parts:
- removed C? (x2): 15pF, symbol agg-kicad:C
- removed C? (x2): 33pF, symbol agg-kicad:C
- removed R?: 1M, symbol agg-kicad:R
- added C1, C6: 47uf/16v, symbol agg-kicad:CP
- added C2, C3: 33pF, symbol agg-kicad:C
- added C5: CP, symbol agg-kicad:CP
- added C8, C9: 15pF, symbol agg-kicad:C
- added CONN-1: CONN_01x04, symbol agg-kicad:CONN_01x04
- added CONN-10: CONN_01x02, symbol agg-kicad:CONN_01x02
- added CONN-6: CONN_01x06, symbol agg-kicad:CONN_01x06
- added CONN-9: CONN_01x11, symbol agg-kicad:CONN_01x11
- added R10, R11, R9: 27R, symbol agg-kicad:R
- added R14: 1M, symbol agg-kicad:R
- added R15, R16, R17: 1K, symbol agg-kicad:R
- added R3: 3K3, symbol agg-kicad:R
- added R6, R7: 330R, symbol agg-kicad:R
- C100: value 470uf/10v -> 470uf/6.3v
- C101: value 1000uf/6.3v -> 4700uf/6.3v
- gave numbers to parts that had none: 2
Connections:
- net labels added: AD0, AD1, AD2, AD3, AD4, AD5, AD6, AD7, B-Y_OUT, IC12_Eb, PrinterPortClk, PrinterPortPin10, PrinterPortPin3, R-Y_OUT, RD0, RD1, RD2, RD3, RD4, RD5, RD6, RD7, V_CAS_, V_RAS_, V_RW_, Y_OUT, ~8255_ENABLE, ~CAS0, ~CAS1, ~RAS, ~VDP_INT
- net labels removed: NC, ~MERQ
- wire segments 275 -> 435
- no-connect marks 1 -> 3
Other:
- note added: "(LLL) wires to P913\nin 4CEC PCB"
- note added: "(RRR) wires to P917\nin AV input PCB (+slot switch)"
- note added: "(UUU) wires to P902\nin front PCB"
- note added: "(WWW) wires to P914\nin AV input PCB"
- note added: "(XXX) wires to AV input PCB\n(Printer port)"
- note added: "LOAD BUTTON"
- note added: "RESET BUTTON"
- note added: "RUN BUTTON"
- moved on the sheet: IC1, IC12, IC13, IC14, IC16, IC24, IC25A, IC25B, IC25C, IC25D, IC25E, IC25F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

Commit message: Add files via upload
Connections:
- net labels added: PrinterPort_BUSY, PrinterPort_~PSTB
- net labels removed: PrinterPortPin10, PrinterPortPin3
Other:
- note added: "PDB0"
- note added: "PDB1"
- note added: "PDB2"
- note added: "PDB3"
- note added: "PDB4"
- note added: "PDB5"
- note added: "PDB6"
- note added: "PDB7"
- note added: "PPort-1"
- note added: "PPort-11"
- note added: "PPort-14"
- note added: "PPort-2"
- note added: "PPort-3"
- note added: "PPort-4"
- note added: "PPort-5"
- note added: "PPort-6"
- note added: "PPort-7"
- note added: "PPort-8"
- note added: "PPort-9"
- note added: "~PSTB"
Changed lines of the file:
@@
 U 1 1 66E82009
 P -240 9820
-F 0 "CONN-9" H -550 9690 50  0000 C CNN
-F 1 "CONN_01x11" V -454 9315 50  0000 C CNN
+F 0 "CONN-9" H -290 8670 50  0000 C CNN
+F 1 "CONN_01x11" H -400 8510 50  0000 C CNN
 F 2 "" H -240 9820 50  0001 C CNN
 F 3 "" H -240 9820 50  0001 C CNN
@@
 Text Notes 660  7270 0    51   ~ 0
 (RRR) wires to P917\nin AV input PCB (+slot switch)
-Text Notes -500 8460 3    51   ~ 0
+Text Notes -1240 10080 0    51   ~ 0
 (XXX) wires to AV input PCB\n(Printer port)
 Text Notes 4420 11100 0    51   ~ 0
@@
 Text GLabel 2030 9930 2    51   Input ~ 0
 PrinterPortClk
+Text GLabel 2030 9130 2    51   Input ~ 0
+D0
+Text GLabel 2030 9630 2    51   Input ~ 0
+D1
+Text GLabel 2030 9530 2    51   Input ~ 0
+D2
+Text GLabel 2030 9230 2    51   Input ~ 0
+D3
+Text GLabel 2030 9330 2    51   Input ~ 0
+D4
+Text GLabel 2030 9430 2    51   Input ~ 0
+D5
 Text GLabel 2030 9030 2    51   Input ~ 0
-D0
-Text GLabel 2030 9130 2    51   Input ~ 0
-D1
-Text GLabel 2030 9230 2    51   Input ~ 0
-D2
-Text GLabel 2030 9330 2    51   Input ~ 0
-D3
-Text GLabel 2030 9430 2    51   Input ~ 0
-D4
-Text GLabel 2030 9530 2    51   Input ~ 0
-D5
-Text GLabel 2030 9630 2    51   Input ~ 0
 D6
 Text GLabel 2030 9730 2    51   Input ~ 0
 D7
 Text GLabel 6160 4530 1    51   Input ~ 0
-PrinterPortPin3
+PrinterPort_~PSTB
 Text GLabel -80  9620 3    51   Input ~ 0
-PrinterPortPin3
+PrinterPort_~PSTB
 Wire Wire Line
 	-140 9620 -80  9620
 Text GLabel 7960 6380 2    51   Input ~ 0
-PrinterPortPin10
+PrinterPort_BUSY
 Text GLabel -80  8920 1    51   Input ~ 0
-PrinterPortPin10
+PrinterPort_BUSY
 Wire Wire Line
 	-140 8920 -80  8920
+Text Notes -700 8820 0    51   ~ 0
+PPort-14
+Text Notes -700 8930 0    51   ~ 0
+PPort-11
+Text Notes -700 9030 0    51   ~ 0
+PPort-7
+Text Notes -700 9130 0    51   ~ 0
+PPort-6
+Text Notes -700 9230 0    51   ~ 0
+PPort-5
+Text Notes -700 9320 0    51   ~ 0
+PPort-4
+Text Notes -700 9420 0    51   ~ 0
+PPort-3
+Text Notes -700 9520 0    51   ~ 0
+PPort-2
+Text Notes -700 9620 0    51   ~ 0
+PPort-1
+Text Notes -700 9720 0    51   ~ 0
+PPort-9
+Text Notes -700 9830 0    51   ~ 0
+PPort-8
+Text Notes -980 9520 0    51   ~ 0
+PDB0
+Text Notes -970 9620 0    51   ~ 0
+~PSTB
+Text Notes -970 9730 0    51   ~ 0
+PDB7
+Text Notes -980 9830 0    51   ~ 0
+PDB6
+Text Notes -990 9410 0    51   ~ 0
+PDB1
+Text Notes -990 9310 0    51   ~ 0
+PDB2
+Text Notes -970 9230 0    51   ~ 0
+PDB3
+Text Notes -1000 9140 0    51   ~ 0
+PDB4
+Text Notes -990 9040 0    51   ~ 0
+PDB5
 $EndSCHEMATC

Commit message: Add files via upload
Parts:
- added CONN-1/CONN-5: Conn_02x11_Top_Bottom, symbol Connector_Generic:Conn_02x11_Top_Bottom
- added KEYBOARDCONN-0: external MALE connector, symbol Connector_Generic:Conn_02x11_Top_Bottom
- added R26, R27: 10K, symbol agg-kicad:R
- added TR1, TR2: A733_PNP_BCE, symbol Device:Q_PNP_BCE
- gave numbers to parts that had none: 3
Connections:
- net labels added: CAPS_LED, CAPS_POWER, DRAM_A0, DRAM_A1, DRAM_A2, DRAM_A3, DRAM_A4, DRAM_A5, DRAM_A6, DRAM_A7, DRAM_A7_SEL, DRAM_ADDR_SEL, KANA_LED, KANA_POWER, LOAD_BUTTON_1, LOAD_BUTTON_2, RESET_BUTTON_1, RESET_BUTTON_2, RUN_BUTTON_1, RUN_BUTTON_2, SND_CLK, X0, X1, X2, X3, X4, X5, X6, X7, Y0, Y1, Y2, Y3, Y4, Y5, Y6, Y7, Y8
- net labels removed: IC12_Eb
- wire segments 435 -> 528
- no-connect marks 3 -> 5
Other:
- note added: "CONN-11\n CONN-5"
- note added: "actual keyboard connector"
- note added: "pin header in pcb,\nviewed from component side,\nwires to \nkeyboard connector"
- moved on the sheet: CONN-6, IC1, IC12, IC13, IC14, IC2, IC25C, IC26A, IC26B, IC3, IC4, R2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

Commit message: Add files via upload
Parts:
- added CONN-7: CONN_01x05, symbol agg-kicad:CONN_01x05
- added IC14: HIC-1, symbol agg-kicad:CONN_01x12
- added K?: DIPxx-1Cxx-51x, Relay_THT:Relay_StandexMeder_DIP_LowProfile, symbol Relay:DIPxx-1Cxx-51x
- added R12: 3K3, symbol agg-kicad:R
- added R19, R20, R26: 10K, symbol agg-kicad:R
- added R28: 100, symbol agg-kicad:R
Connections:
- net labels added: BIT_0_-_3, BIT_4_-_7, LOAD_BUTTON_IC13_ENABLE, LOAD_BUTTON_PC3, PC0, PC1, PC2, PC3, RUN_BUTTON_X1, RUN_BUTTON_Y7, ~PC2
- net labels removed: LOAD_BUTTON_2, RUN_BUTTON_1, RUN_BUTTON_2
- wire segments 528 -> 547
- no-connect marks 5 -> 10
Other:
- note added: "LOAD button connects\n8255 PC3 line to this IC13"
- note added: "LOAD button presses:\n-X0+X6 down when Y6 line scanned (so shift+F3 = cload " )\n-X5+X7 down when Y7 line scanned (so Backspace + Return)\nNOTE! MSX1 bios must be scanning keys always rows at ascending order."
- note added: "RUN button presses X1 down when Y7 line scanned\n->F5 function key"
- note added: "to Cassette port"
- moved on the sheet: C1, C100, C101, C2, C3, C5, C6, C7, C8, C9, CONN-1, CONN-1/CONN-5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

Commit message: msx pcb complete, except cassette port related
Parts:
- removed R?: 100R, symbol agg-kicad:R
- R28: value 100 -> 100R
- renumbered R12 to R3
Connections:
- net labels added: PSG_IOA0, PSG_IOA1, PSG_IOA2, PSG_IOA3, PSG_IOA4, PSG_IOA5, PSG_IOB0, PSG_IOB1, PSG_IOB2, PSG_IOB3, PSG_IOB4, PSG_IOB5, PSG_IOB6, ReadBits
- wire segments 547 -> 580
- no-connect marks 10 -> 25
Other:
- moved on the sheet: C7, R12, R18, R20, R23, R28, R3

Commit message: shuold be now final
Parts:
- removed K?: DIPxx-1Cxx-51x, Relay_THT:Relay_StandexMeder_DIP_LowProfile, symbol Relay:DIPxx-1Cxx-51x
- removed R19, R26: 10K, symbol agg-kicad:R
- C5, C7: value CP -> 10uf/16v
Connections:
- net labels added: 8255_RESET, PC4, PC5, PSG_IOA7
- net labels removed: RESET_BUTTON_1, RESET_BUTTON_2
- wire segments 580 -> 609
- no-connect marks 25 -> 21
Other:
- note added: "relay pins \nfrom solder side"
- moved on the sheet: CONN-6, CONN-7, IC13, IC14

Commit message: added filter caps and relay symbol for MSX pcb
Parts:
- added C10, C12, C14, C15, C16, C17, C18, C19, C20, C21, C22, C23, C24, C25, C26, C27, C28, C29, C30, C31, C32, C33, C34, C35, C36: 10nF, symbol agg-kicad:C
- added RL-1: MZ_TAKAMISAWA, Relay_THT:Relay_SPDT_HsinDa_Y14, symbol Relay:MZ_TAKAMISAWA
- renumbered CONN-1 to CON-1, CONN-1/CONN-5 to CON-1/CON-5, CONN-6 to CON-6, CONN-7 to CON-7, CONN-9 to CON-9
Connections:
- wire segments 609 -> 702
- no-connect marks 21 -> 22
Other:
- note added: "1"
- note added: "2"
- note added: "3"
- note added: "4"
- note added: "5"
- note added: "CON-11\n CON-5"
- note added: "CON-7 <-> Cassette port DIN-8\n3 1,2,3,8 GND\n1 4 CMT OUT\n4 5 CMT IN\n2 6 REM+\n5 7 REM-"
- note added: "Filter caps in pcb:"
- note added: "Original PCB had direct 5v line to cartridge port,\nbut now there is this two caps+ coil added between"
- note added: "POWER INPUT"
- note added: "There is also black thick wire soldered to 5V line \nat the solder side of this MSX PCB.\nThis wire comes directly from the 5V source\nin main PCB ( from Q505 leg)."
- note added: "markins on relay:\nMZ\nTAKAMISAWA\nELECTRIC CO. LTD."
- note added: "o"
- note removed: "CONN-11\n CONN-5"
- note removed: "relay pins \nfrom solder side"
- moved on the sheet: C1, CON-1
